File: turbocharge.sch (EAGLE design)
At the start: 69 parts, among them Q01 NMOS40V_10A, Q03 NMOS40V_10A, Q11 PMOS30V_11A, Q12 PMOS30V_11A, Q13 2PMOS30V_2A, Q15 PMOS30V_11A, Q16 PMOS30V_11A, Q21 PMOS30V_11A, Q22 PMOS30V_11A, Q23 PMOS30V_11A, Q25 PMOS30V_11A, Q26 PMOS30V_11A, Q27 PMOS30V_11A, Q28 PMOS30V_11A, Q31 PMOS30V_11A, Q32 PMOS30V_11A, Q33 PMOS30V_11A, Q34 PMOS30V_11A, Q35 PMOS30V_11A, Q36 PMOS30V_11A, Q37 PMOS30V_11A, Q38 PMOS30V_11A, Q41 PMOS30V_11A, Q42 PMOS30V_11A, Q43 PMOS30V_11A, Q44 PMOS30V_11A, Q45 PMOS30V_11A, Q46 PMOS30V_11A, Q47 PMOS30V_11A, Q48 PMOS30V_11A, Q51 PMOS30V_11A, Q52 PMOS30V_11A, Q53 PMOS30V_11A, Q54 PMOS30V_11A, Q55 PMOS30V_11A, Q56 PMOS30V_11A, Q57 PMOS30V_11A, Q58 PMOS30V_11A, Q62 PMOS30V_11A, Q64 PMOS30V_11A, Q66 PMOS30V_11A, Q68 PMOS30V_11A, U1 ATTINY13A10M1, U2 DG408DVZ, U3 CCR20MA_45V

Commit message: .
Parts:
- removed D4, DG1: 4DSCH30V_0A1, dubec:4DSCH30V_0A1
- removed R11, R12: RES100K_16, dubec:RES100K_16
- added D6: 3D_SCHOTTKY30V_0.35V, dubec:3D_SCHOTTKY30V_0.35V
- added Q17: 2PMOS50V_0.17A, dubec:2PMOS50V_0.17A
- added RG11, RG21-: RES100K_16, dubec:RES100K_16
- D2: value 3D_SCHOTTKY30V_0.35V -> 4DSCH30V_0A1; device dubec:3D_SCHOTTKY30V_0.35V -> dubec:4DSCH30V_0A1
- Q11, Q12, Q23: value PMOS30V_11A -> NMOS40V_10A; device dubec:PMOS30V_11A -> dubec:NMOS40V_10A
- Q13: value 2PMOS30V_2A -> NMOS40V_10A; device dubec:2PMOS30V_2A -> dubec:NMOS40V_10A
- renumbered RG21 to RG21+, U$2 to T1
Connections:
- removed net G21: D3.C2, DG1G$2.C, Q21.G, Q22.G, Q23.G, RG21+.2, U2.S3
- removed net N$17: Q12.G, Q13G$1.D, R12.2
- removed net N$18: DG1G$1.A, DG1G$2.A, Q11.G
- new net C4+: D1G$1.C, D1G$2.C, D1G$3.C, D1G$4.A, Q17G$1.S, RG11.1
- new net G21+: D3.C2, Q17G$1.G, Q21.G, Q22.G, RG21+.2, U2.S3
- new net G21-: Q01.G, Q17G$1.D, Q23.G, RG21-.2
- new net S+11: Q11.S, Q12.S
- net BATT+: now also D2G$3.C, D2G$4.C; no longer D1G$1.C, D1G$2.C, D1G$3.C, D4G$3.C
- net BATT-: now also Q13.S, RG21-.1; no longer Q01.S, R12.1
- net C1: now also Q17G$2.S, Q23.D; no longer Q13G$1.S, Q13G$2.S
- net C2: no longer R11.1
- net C5: now also D2G$4.A; no longer D1G$4.A
- net C6: now also D2G$3.A; no longer D4G$3.A
- net G02: now also Q17G$2.D; no longer Q13G$2.D
- net G11: now also Q11.G, Q12.G, Q13.G, RG11.2; no longer DG1G$1.C, Q01.G, Q13G$1.G, R11.2
- net G13: now also Q17G$2.G; no longer Q13G$2.G
- net G41: now also D6.C3; no longer D2.C3
- net G51: now also D6.C2; no longer D2.C2
- net G61: now also D6.C1; no longer D2.C1
- net N$12: now also D6.A2; no longer D2.A2
- net N$13: now also D6.A3; no longer D2.A3
- net N$8: now also D6.A1; no longer D2.A1
- net S+: now also D2G$1.A, D2G$2.A; no longer D4G$1.A, D4G$2.A
- net S-: now also Q13.D; no longer Q23.D
- net S-21: now also Q01.S; no longer Q11.S, Q12.S
- net VCC: now also D2G$1.C, D2G$2.C; no longer D4G$1.C, D4G$2.C
Other:
- moved on the sheet: D1G$1, D1G$2, D1G$3, D1G$4, R1

Commit message: .
Other:
- moved on the sheet: Q01, Q11, Q12, Q13, Q21, Q22, Q23, Q33, Q34, Q41, Q42, Q51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

Commit message: .
Parts:
- removed D3, D6: 3D_SCHOTTKY30V_0.35V, dubec:3D_SCHOTTKY30V_0.35V
- removed Q03: NMOS40V_10A, dubec:NMOS40V_10A
- removed Q15: PMOS30V_11A, dubec:PMOS30V_11A
- removed Q17: 2PMOS50V_0.17A, dubec:2PMOS50V_0.17A
- removed R7, RG11, RG21+, RG21-, RG31, RG41, RG51, RG61: RES100K_16, dubec:RES100K_16
- removed U2: DG408DVZ, dubec:DG408DVZ
- added Q1, Q18, Q2: NMOS40V_10A, dubec:NMOS40V_10A
- added RGS+2, RGS-2, RGS1, RGS3, RGS4, RGS5, RGS6, RGT+2, RGT-2, RGT1, RGT3, RGT4, RGT5, RGT6: RES100K_16, dubec:RES100K_16
- added U$2, U$3, U$4, U$5, U$6, U$7, U4: 2NMOS30V_0.1A, dubec:2NMOS30V_0.1A
- Q16: value PMOS30V_11A -> 2PMOS50V_0.17A; device dubec:PMOS30V_11A -> dubec:2PMOS50V_0.17A
- Q27, Q28: value PMOS30V_11A -> NMOS40V_10A; device dubec:PMOS30V_11A -> dubec:NMOS40V_10A
- renumbered Q01 to Q24, Q13 to Q14
Connections:
- net S+11 renamed SS+1
- net S+21 renamed SS+2
- net S+22 renamed ST+2
- net S+31 renamed SS+3
- net S+32 renamed ST+3
- net S+41 renamed SS+4
- net S+42 renamed ST+4
- net S+51 renamed SS+5
- net S+52 renamed ST+5
- net S-21 renamed SS-2
- net S-22 renamed ST-2
- net S-31 renamed SS-3
- net S-32 renamed ST-3
- net S-41 renamed SS-4
- net S-42 renamed ST-4
- net S-51 renamed SS-5
- net S-52 renamed ST-5
- removed net G02: Q03.G, Q17G$2.D, R7.2
- removed net G11: D3.C3, Q11.G, Q12.G, Q14.G, RG11.2, U2.S2
- removed net G13: Q15.G, Q16.G, Q17G$2.G
- removed net G21+: D3.C2, Q17G$1.G, Q21.G, Q22.G, RG21+.2, U2.S3
- removed net G21-: Q17G$1.D, Q23.G, Q24.G, RG21-.2
- removed net G22: Q25.G, Q26.G, Q27.G, Q28.G
- removed net G31: D3.C1, Q31.G, Q32.G, Q33.G, Q34.G, RG31.2, U2.S4
- removed net G32: Q35.G, Q36.G, Q37.G, Q38.G
- removed net G41: D6.C3, Q41.G, Q42.G, Q43.G, Q44.G, RG41.2, U2.S5
- removed net G42: Q45.G, Q46.G, Q47.G, Q48.G
- removed net G51: D6.C2, Q51.G, Q52.G, Q53.G, Q54.G, RG51.2, U2.S6
- removed net G52: Q55.G, Q56.G, Q57.G, Q58.G
- removed net G61: D6.C1, Q62.G, Q64.G, RG61.2, U2.S7
- removed net G62: Q66.G, Q68.G
- removed net N$10: U2.A1
- removed net N$11: U2.A0
- removed net N$12: D51.C, D6.A2
- removed net N$8: D6.A1, D61.C
- removed net N$9: U2.A2
- removed net S+12: Q15.S, Q16.S
- new net !EN_S1: U4G$2.G
- new net EN_S2: U4G$1.G
- new net EN_S3: U$2G$1.G
- new net EN_S4: U$2G$2.G
- new net EN_S5: U$3G$1.G
- new net EN_S6: U$3G$2.G
- new net EN_T1: U$4G$1.G
- new net EN_T2: U$4G$2.G, U$5G$1.G
- new net EN_T3: U$5G$2.G
- new net EN_T4: U$6G$1.G
- new net EN_T5: U$6G$2.G
- new net EN_T6: U$7G$1.G
- new net GS+2: Q16G$1.G, Q21.G, Q22.G, RGS+2.2, U4G$1.D
- new net GS-2: Q16G$1.D, Q23.G, Q24.G, RGS-2.2
- new net GS1: Q11.G, Q12.G, Q14.G, RGS1.2, U4G$2.D
- new net GS3: Q31.G, Q32.G, Q33.G, Q34.G, RGS3.2, U$2G$1.D
- new net GS4: Q41.G, Q42.G, Q43.G, Q44.G, RGS4.2, U$2G$2.D
- new net GS5: Q51.G, Q52.G, Q53.G, Q54.G, RGS5.2, U$3G$1.D
- new net GS6: Q62.G, Q64.G, RGS6.2, U$3G$2.D
- new net GT+2: Q25.G, Q26.G, RGT+2.2, U$5G$1.D
- new net GT-2: Q27.G, Q28.G, RGT-2.2, U$4G$2.S
- new net GT1: Q1.G, Q18.G, Q2.G, RGT1.2, U$4G$1.S
- new net GT3: Q35.G, Q36.G, Q37.G, Q38.G, RGT3.2, U$5G$2.D
- new net GT4: Q45.G, Q46.G, Q47.G, Q48.G, RGT4.2, U$6G$1.D
- new net GT5: Q55.G, Q56.G, Q57.G, Q58.G, RGT5.2, U$6G$2.D
- new net GT6: Q66.G, Q68.G, RGT6.2, U$7G$1.D
- new net ST+1: Q1.S, Q2.S
- net BATT+: now also RGS+2.1, RGS3.1, RGS4.1, RGS5.1, RGS6.1, RGT+2.1, RGT3.1, RGT4.1, RGT5.1, RGT6.1; no longer RG21+.1, RG31.1, RG41.1, RG51.1, RG61.1, U2.V+
- net BATT-: now also Q18.S, RGS-2.1, RGT-2.1, RGT1.1, U$2G$1.S, U$2G$2.S, U$3G$1.S, U$3G$2.S, U$5G$1.S, U$5G$2.S, U$6G$1.S, U$6G$2.S, U$7G$1.S, U4G$1.S, U4G$2.S; no longer Q03.S, R7.1, RG21-.1, U2.S1
- net C1: now also Q1.D; no longer Q15.D, Q17G$2.S
- net C4+: now also Q16G$1.S, RGS1.1, U$4G$1.D, U$4G$2.D; no longer Q17G$1.S, RG11.1
- net N$13: no longer D6.A3
- net N$14: no longer D3.A1
- net N$15: no longer D3.A2
- net N$16: no longer D3.A3
- net T+: now also Q2.D; no longer Q16.D
- net T-: now also Q18.D; no longer Q03.D
- net VCC: no longer U2.EN
Other:
- moved on the sheet: D1G$1, D1G$2, D1G$3, D1G$4, D2G$1, D2G$2, D2G$3, D2G$4, Q16G$1, Q25, Q26, Q27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

Commit message: Switching back to an analog switch
Parts:
- removed U3: CCR20MA_45V, dubec:CCR20MA_45V
- added C1: (no value), dubec:CAP47UF_10V
- added R3, R4: RES4.7K_16, dubec:RES4.7K_16
- added R5: RES01_0.75W, dubec:RES01_0.75W
- added U$8: NMOS30V_30A, dubec:NMOS30V_30A
- added U10: CCR20MA_45V, dubec:CCR20MA_45V
- added U2: TC1240A, dubec:TC1240A
- added U5, U6: 74HC595, dubec:74HC595
- U1: value ATTINY13A10M1 -> LT3757IDD; device dubec:ATTINY13A10M1 -> dubec:LT3757IDD
Connections:
- removed net N$6: U1.PB1
- new net !OE: R3.2, U5.!OE, U6.!OE
- new net !RESET: R4.2, U5.!MR, U6.!MR
- new net CP: U5.SHCP, U5.STCP, U6.SHCP, U6.STCP
- new net DSS: U5.DS
- new net DST: U5.Q7S, U6.DS
- new net FBX: U1.FBX
- new net N$10: T1.5, T1.7, U$8.D
- new net N$11: U1.!SHDN, U1.INTVCC, U1.VIN, U2.VOUT
- new net N$19: U6.Q7S
- new net N$20: U5.Q7
- new net N$8: C1.2, U2.C+
- new net N$9: C1.1, U2.C-
- new net T~: T1.2
- net !EN_S1: now also U5.Q0
- net BATT-: now also R4.1, U$1.C, U5.GND, U6.GND
- net C1: now also D2G$1.A, D2G$2.A, U10.A; no longer U3.A
- net EN_S2: now also U5.Q1
- net EN_S3: now also U5.Q2
- net EN_S4: now also U5.Q3
- net EN_S5: now also U5.Q4
- net EN_S6: now also U5.Q5
- net EN_T1: now also U6.Q0
- net EN_T2: now also U6.Q1
- net EN_T3: now also U6.Q2
- net EN_T4: now also U6.Q3
- net EN_T5: now also U6.Q4
- net EN_T6: now also U6.Q5
- net N$1: now also U6.Q7; no longer U1.PB4
- net N$2: now also U5.Q6; no longer U1.PB3
- net N$3: now also U6.Q6; no longer U1.PB5
- net N$4: now also U10.C; no longer U3.C
- net N$5: now also U$8.G, U1.GATE; no longer U1.PB2
- net N$7: now also R5.2, U$8.S, U1.SENSE; no longer U1.PB0
- net S+: now also T1.6, T1.8, U2.VIN; no longer D2G$1.A, D2G$2.A
- net S-: now also R5.1, U1.SYNC, U2.GND, U2.SHDN; no longer U$1.C
- net T-: now also T1.1, T1.3
- net VCC: now also R3.1, U5.VCC, U6.VCC; no longer U1.VCC
Other:
- note added: "Battery refd"
- note added: "Routing"
- note added: "Source refd"
- moved on the sheet: D11, D1G$1, D1G$2, D1G$3, D1G$4, D21, D2G$1, D2G$2, D2G$3, D2G$4, D31, D41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

Commit message: Analog switches are back
Parts:
- removed U$2, U$3, U$4, U$5, U$6, U$7: 2NMOS30V_0.1A, dubec:2NMOS30V_0.1A
- removed U6: 74HC595, dubec:74HC595
- added Q15: NMOS40V_10A, dubec:NMOS40V_10A
- added Q3: 2PMOS50V_0.17A, dubec:2PMOS50V_0.17A
- added U3: 74HC595, dubec:74HC595
- Q1: value NMOS40V_10A -> 2NMOS30V_0.1A; device dubec:NMOS40V_10A -> dubec:2NMOS30V_0.1A
- Q16: value 2PMOS50V_0.17A -> NMOS40V_10A; device dubec:2PMOS50V_0.17A -> dubec:NMOS40V_10A
- Q2: value NMOS40V_10A -> 2PMOS50V_0.17A; device dubec:NMOS40V_10A -> dubec:2PMOS50V_0.17A
- U1: value LT3757IDD -> DG508BEN-T1-GE4; device dubec:LT3757IDD -> dubec:DG508BEN-T1-GE4
- U2: value TC1240A -> DG508BEN-T1-GE4; device dubec:TC1240A -> dubec:DG508BEN-T1-GE4
- U4: value 2NMOS30V_0.1A -> LT3757IDD; device dubec:2NMOS30V_0.1A -> dubec:LT3757IDD
- U5: value 74HC595 -> TC1240A; device dubec:74HC595 -> dubec:TC1240A
Connections:
- removed net !RESET: R4.2, U5.!MR, U6.!MR
- removed net DSS: U5.DS
- removed net DST: U5.Q7S, U6.DS
- removed net EN_S2: U4G$1.G, U5.Q1
- removed net EN_S3: U$2G$1.G, U5.Q2
- removed net EN_S4: U$2G$2.G, U5.Q3
- removed net EN_S5: U$3G$1.G, U5.Q4
- removed net EN_S6: U$3G$2.G, U5.Q5
- removed net EN_T1: U$4G$1.G, U6.Q0
- removed net EN_T2: U$4G$2.G, U$5G$1.G, U6.Q1
- removed net EN_T3: U$5G$2.G, U6.Q2
- removed net EN_T4: U$6G$1.G, U6.Q3
- removed net EN_T5: U$6G$2.G, U6.Q4
- removed net EN_T6: U$7G$1.G, U6.Q5
- removed net N$20: U5.Q7
- removed net N$3: U6.Q6
- new net AS0: U1.A0, U3.Q1
- new net AS1: U1.A1, U3.Q2
- new net AS2: U1.A2, U3.Q3
- new net AT0: U2.A0, U3.Q4
- new net AT1: U2.A1, U3.Q5
- new net AT2: U2.A2, U3.Q6
- new net DS: U3.DS
- new net N$23: Q3G$1.G, U2.S2
- net !EN_S1: now also Q1G$2.G, U1.EN, U3.Q0; no longer U4G$2.G, U5.Q0
- net !OE: now also U3.!OE; no longer U5.!OE, U6.!OE
- net BATT+: now also U1.V+, U2.EN, U2.V+
- net BATT-: now also Q1G$2.S, U1.D, U1.V-, U2.D, U2.S1, U2.V-; no longer R4.1, U$1.C, U$2G$1.S, U$2G$2.S, U$3G$1.S, U$3G$2.S, U$5G$1.S, U$5G$2.S, U$6G$1.S, U$6G$2.S, U$7G$1.S, U4G$1.S, U4G$2.S, U5.GND, U6.GND
- net C1: now also Q15.D; no longer D2G$1.A, D2G$2.A, Q1.D
- net C4+: now also Q2G$1.S, Q3G$1.S, Q3G$2.S; no longer Q16G$1.S, U$4G$1.D, U$4G$2.D
- net CP: now also U3.SHCP, U3.STCP; no longer U5.SHCP, U5.STCP, U6.SHCP, U6.STCP
- net FBX: now also U4.FBX; no longer U1.FBX
- net GS+2: now also Q2G$1.G, U1.S1; no longer Q16G$1.G, U4G$1.D
- net GS-2: now also Q2G$1.D; no longer Q16G$1.D
- net GS1: now also Q1G$2.D; no longer U4G$2.D
- net GS3: now also U1.S2; no longer U$2G$1.D
- net GS4: now also U1.S3; no longer U$2G$2.D
- net GS5: now also U1.S4; no longer U$3G$1.D
- net GS6: now also U1.S5, U1.S6, U1.S7, U1.S8; no longer U$3G$2.D
- net GT+2: now also Q3G$2.G, U2.S3; no longer U$5G$1.D
- net GT-2: now also Q3G$2.D; no longer U$4G$2.S
- net GT1: now also Q15.G, Q16.G, Q3G$1.D; no longer Q1.G, Q2.G, U$4G$1.S
- net GT3: now also U2.S4; no longer U$5G$2.D
- net GT4: now also U2.S5; no longer U$6G$1.D
- net GT5: now also U2.S6; no longer U$6G$2.D
- net GT6: now also U2.S7, U2.S8; no longer U$7G$1.D
- net N$1: now also U3.Q7; no longer U6.Q7
- net N$11: now also U4.!SHDN, U4.INTVCC, U4.VIN, U5.VOUT; no longer U1.!SHDN, U1.INTVCC, U1.VIN, U2.VOUT
- net N$19: now also U3.Q7S; no longer U6.Q7S
- net N$2: now also R4.2, U3.!MR; no longer U5.Q6
- net N$5: now also U4.GATE; no longer U1.GATE
- net N$7: now also U4.SENSE; no longer U1.SENSE
- net N$8: now also U5.C+; no longer U2.C+
- net N$9: now also U5.C-; no longer U2.C-
- net S+: now also D2G$1.A, D2G$2.A, U5.VIN; no longer U2.VIN
- net S-: now also R4.1, U$1.C, U3.GND, U4.GND, U4.SYNC, U5.GND, U5.SHDN; no longer U1.SYNC, U2.SHDN
- net ST+1: now also Q15.S, Q16.S; no longer Q1.S, Q2.S
- net T+: now also Q16.D; no longer Q2.D
- net VCC: now also U3.VCC; no longer U5.VCC, U6.VCC
Other:
- note added: "Pick-N-Place Hell"
- note added: "Reception of the Electric Potential Hell"
- note removed: "Battery refd"
- note removed: "Routing"
- note removed: "Source refd"
- moved on the sheet: C1, D11, D1G$1, D1G$2, D1G$3, D1G$4, D21, D2G$1, D2G$2, D2G$3, D2G$4, D31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

Commit message: Composing the schematic
Parts:
- added C2: CAP47UF_10V, dubec:CAP47UF_10V
- added C3: CAP47NF_16V, dubec:CAP47NF_16V
- added C4: CAP22N_50V, dubec:CAP22N_50V
- added C5: CAP220U_6V3, dubec:CAP220U_6V3
- added R6: RES41.2K_16, dubec:RES41.2K_16
- added R7: RES6.8K_16, dubec:RES6.8K_16
- added R8: RES2.2K_16, dubec:RES2.2K_16
- C1: value (none) -> CAP47UF_10V
Connections:
- removed net N$11: U4.!SHDN, U4.INTVCC, U4.VIN, U5.VOUT
- new net N$12: R7.2, U4.VC
- new net N$17: C4.2, R7.1
- new net N$3: R6.2, U4.RT
- new net N$6: C3.2, U4.SS
- new net VCC_REG: C2.2, U4.!SHDN, U4.INTVCC, U4.VIN, U5.VOUT
- net BATT-: now also U2.S8
- net FBX: now also R8.2
- net GT6: no longer U2.S8
- net S+: now also C5.2
- net S-: now also C2.1, C3.1, C4.1, C5.1, R6.1, R8.1
Other:
- moved on the sheet: C1, R3, R4, R5, T1, U$8, U3, U4, U5
