File: lipolski.brd (EAGLE design)
At the start: 56.2 x 21 mm, 90 parts, among them Q1 2NMOS30V_0.1A, Q11 NMOS40V_10A, Q12 NMOS40V_10A, Q14 NMOS40V_10A, Q15 NMOS40V_10A, Q16 NMOS40V_10A, Q18 NMOS40V_10A, Q2 2PMOS50V_0.17A, Q21 PMOS30V_11A, Q22 PMOS30V_11A, Q23 NMOS40V_10A, Q24 NMOS40V_10A, Q25 PMOS30V_11A, Q26 PMOS30V_11A, Q27 NMOS40V_10A, Q28 NMOS40V_10A, Q3 2PMOS50V_0.17A, Q31 PMOS30V_11A, Q32 PMOS30V_11A, Q33 PMOS30V_11A, Q34 PMOS30V_11A, Q35 PMOS30V_11A, Q36 PMOS30V_11A, Q37 PMOS30V_11A, Q38 PMOS30V_11A, Q41 PMOS30V_11A, Q42 PMOS30V_11A, Q43 PMOS30V_11A, Q44 PMOS30V_11A, Q45 PMOS30V_11A, Q46 PMOS30V_11A, Q47 PMOS30V_11A, Q48 PMOS30V_11A, Q51 PMOS30V_11A, Q52 PMOS30V_11A, Q53 PMOS30V_11A, Q54 PMOS30V_11A, Q55 PMOS30V_11A, Q56 PMOS30V_11A, Q57 PMOS30V_11A, Q58 PMOS30V_11A, Q62 PMOS30V_11A, Q64 PMOS30V_11A, Q66 PMOS30V_11A, Q68 PMOS30V_11A, T1 TFORM_4_4311_4A4, U1 DG508BEN-T1-GE4, U10 CCR20MA_45V, U2 DG508BEN-T1-GE4, U3 74HC595, U4 LT3757IDD, U5 TC1240A

Commit message: LTC3803 simu
Parts:
- moved C1 49.1 mm to (29.6, 29.6)
- moved C2 49.1 mm to (33.2, 29.6)
- moved C5 49.1 mm to (25.2, 31.8)
- moved R8 49.1 mm to (24.0, 26.2)
Changed lines of the file:
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@@
 <attribute name="TEMP" value="X7R" x="36.8" y="23" size="1.778" layer="27" display="off"/>
 </element>
-<element name="C2" library="dubec" package="0805" value="CAP47UF_10V" x="-3" y="-3.6">
-<attribute name="MANUFACTURER" value="TDK Corporation" x="-3" y="-3.6" size="1.778" layer="27" display="off"/>
-<attribute name="MFG_PART_#" value="C2012X5R1A476M125AC" x="-3" y="-3.6" size="1.778" layer="27" display="off"/>
-<attribute name="TOLERANCE" value="±20%" x="-3" y="-3.6" size="1.778" layer="27" display="off"/>
-<attribute name="DIGIKEY_PART_#" value="445-8239-1-ND" x="-3" y="-3.6" size="1.778" layer="27" display="off"/>
-<attribute name="USD" value="0.93" x="-3" y="-3.6" size="1.778" layer="27" display="off"/>
-<attribute name="TEMP" value="X5R" x="-3" y="-3.6" size="1.778" layer="27" display="off"/>
+<element name="C2" library="dubec" package="0805" value="CAP47UF_10V" x="33.2" y="29.6">
+<attribute name="MANUFACTURER" value="TDK Corporation" x="33.2" y="29.6" size="1.778" layer="27" display="off"/>
+<attribute name="MFG_PART_#" value="C2012X5R1A476M125AC" x="33.2" y="29.6" size="1.778" layer="27" display="off"/>
+<attribute name="TOLERANCE" value="±20%" x="33.2" y="29.6" size="1.778" layer="27" display="off"/>
+<attribute name="DIGIKEY_PART_#" value="445-8239-1-ND" x="33.2" y="29.6" size="1.778" layer="27" display="off"/>
+<attribute name="USD" value="0.93" x="33.2" y="29.6" size="1.778" layer="27" display="off"/>
+<attribute name="TEMP" value="X5R" x="33.2" y="29.6" size="1.778" layer="27" display="off"/>
 </element>
-<element name="C1" library="dubec" package="0805" value="CAP47UF_10V" x="-6.6" y="-3.6">
-<attribute name="MANUFACTURER" value="TDK Corporation" x="-6.6" y="-3.6" size="1.778" layer="27" display="off"/>
-<attribute name="MFG_PART_#" value="C2012X5R1A476M125AC" x="-6.6" y="-3.6" size="1.778" layer="27" display="off"/>
-<attribute name="TOLERANCE" value="±20%" x="-6.6" y="-3.6" size="1.778" layer="27" display="off"/>
-<attribute name="DIGIKEY_PART_#" value="445-8239-1-ND" x="-6.6" y="-3.6" size="1.778" layer="27" display="off"/>
-<attribute name="USD" value="0.93" x="-6.6" y="-3.6" size="1.778" layer="27" display="off"/>
-<attribute name="TEMP" value="X5R" x="-6.6" y="-3.6" size="1.778" layer="27" display="off"/>
+<element name="C1" library="dubec" package="0805" value="CAP47UF_10V" x="29.6" y="29.6">
+<attribute name="MANUFACTURER" value="TDK Corporation" x="29.6" y="29.6" size="1.778" layer="27" display="off"/>
+<attribute name="MFG_PART_#" value="C2012X5R1A476M125AC" x="29.6" y="29.6" size="1.778" layer="27" display="off"/>
+<attribute name="TOLERANCE" value="±20%" x="29.6" y="29.6" size="1.778" layer="27" display="off"/>
+<attribute name="DIGIKEY_PART_#" value="445-8239-1-ND" x="29.6" y="29.6" size="1.778" layer="27" display="off"/>
+<attribute name="USD" value="0.93" x="29.6" y="29.6" size="1.778" layer="27" display="off"/>
+<attribute name="TEMP" value="X5R" x="29.6" y="29.6" size="1.778" layer="27" display="off"/>
 </element>
-<element name="C5" library="dubec" package="1210" value="CAP220U_6V3" x="-11" y="-1.4">
-<attribute name="MANUFACTURER" value="Samsung Electro-Mechanics America, Inc." x="-11" y="-1.4" size="1.778" layer="27" display="off"/>
-<attribute name="EURO" value="20.40/25" x="-11" y="-1.4" size="1.778" layer="27" display="off"/>
-<attribute name="MFG_PART_#" value="CL32A227MQVNNNE" x="-11" y="-1.4" size="1.778" layer="27" display="off"/>
-<attribute name="TOLERANCE" value="±20%" x="-11" y="-1.4" size="1.778" layer="27" display="off"/>
-<attribute name="DIGIKEY_PART_#" value="1276-3375-1-ND" x="-11" y="-1.4" size="1.778" layer="27" display="off"/>
-<attribute name="TEMP" value="X5R, -55°C ~ 85°C" x="-11" y="-1.4" size="1.778" layer="27" display="off"/>
+<element name="C5" library="dubec" package="1210" value="CAP220U_6V3" x="25.2" y="31.8">
+<attribute name="MANUFACTURER" value="Samsung Electro-Mechanics America, Inc." x="25.2" y="31.8" size="1.778" layer="27" display="off"/>
+<attribute name="EURO" value="20.40/25" x="25.2" y="31.8" size="1.778" layer="27" display="off"/>
+<attribute name="MFG_PART_#" value="CL32A227MQVNNNE" x="25.2" y="31.8" size="1.778" layer="27" display="off"/>
+<attribute name="TOLERANCE" value="±20%" x="25.2" y="31.8" size="1.778" layer="27" display="off"/>
+<attribute name="DIGIKEY_PART_#" value="1276-3375-1-ND" x="25.2" y="31.8" size="1.778" layer="27" display="off"/>
+<attribute name="TEMP" value="X5R, -55°C ~ 85°C" x="25.2" y="31.8" size="1.778" layer="27" display="off"/>
 </element>
-<element name="R8" library="dubec" package="0402" value="RES2.2K_16" x="-12.2" y="-7">
-<attribute name="MANUFACTURER" value="Vishay Dale" x="-12.2" y="-7" size="1.778" layer="27" display="off"/>
-<attribute name="MFG_PART_#" value="CRCW04022K20FKED" x="-12.2" y="-7" size="1.778" layer="27" display="off"/>
-<attribute name="TOLERANCE" value="±1%" x="-12.2" y="-7" size="1.778" layer="27" display="off"/>
-<attribute name="DIGIKEY_PART_#" value="541-2.20KLCT-ND" x="-12.2" y="-7" size="1.778" layer="27" display="off"/>
-<attribute name="USD" value="2.11/50" x="-12.2" y="-7" size="1.778" layer="27" display="off"/>
-<attribute name="TEMP" value="±100ppm/°C" x="-12.2" y="-7" size="1.778" layer="27" display="off"/>
+<element name="R8" library="dubec" package="0402" value="RES2.2K_16" x="24" y="26.2">
+<attribute name="MANUFACTURER" value="Vishay Dale" x="24" y="26.2" size="1.778" layer="27" display="off"/>
+<attribute name="MFG_PART_#" value="CRCW04022K20FKED" x="24" y="26.2" size="1.778" layer="27" display="off"/>
+<attribute name="TOLERANCE" value="±1%" x="24" y="26.2" size="1.778" layer="27" display="off"/>
+<attribute name="DIGIKEY_PART_#" value="541-2.20KLCT-ND" x="24" y="26.2" size="1.778" layer="27" display="off"/>
+<attribute name="USD" value="2.11/50" x="24" y="26.2" size="1.778" layer="27" display="off"/>
+<attribute name="TEMP" value="±100ppm/°C" x="24" y="26.2" size="1.778" layer="27" display="off"/>
 </element>
 </elements>
@@
 <wire x1="16.1" y1="2.6" x2="19.375" y2="3" width="0" layer="19" extent="1-1"/>
 <wire x1="35.8" y1="1.85" x2="19.375" y2="3" width="0" layer="19" extent="1-1"/>
-<wire x1="-3.9" y1="-3.6" x2="16.1" y2="2.6" width="0" layer="19" extent="1-1"/>
-<wire x1="-12.4" y1="-1.4" x2="-3.9" y2="-3.6" width="0" layer="19" extent="1-1"/>
-<wire x1="-12.7" y1="-7" x2="-12.4" y2="-1.4" width="0" layer="19" extent="1-1"/>
+<wire x1="32.3" y1="29.6" x2="16.1" y2="2.6" width="0" layer="19" extent="1-1"/>
+<wire x1="23.8" y1="31.8" x2="32.3" y2="29.6" width="0" layer="19" extent="1-1"/>
+<wire x1="23.5" y1="26.2" x2="23.8" y2="31.8" width="0" layer="19" extent="1-1"/>
 </signal>
 <signal name="S+">
@@
 <wire x1="13.975" y1="18" x2="28.65" y2="24.2" width="0" layer="19" extent="1-1"/>
 <wire x1="15.1" y1="2.6" x2="13.975" y2="5.5" width="0" layer="19" extent="1-1"/>
-<wire x1="-9.6" y1="-1.4" x2="13.975" y2="5.5" width="0" layer="19" extent="1-1"/>
+<wire x1="26.6" y1="31.8" x2="13.975" y2="5.5" width="0" layer="19" extent="1-1"/>
 </signal>
 <signal name="BATT-">
@@
 <contactref element="U5" pad="6"/>
 <contactref element="C1" pad="2"/>
-<wire x1="-5.7" y1="-3.6" x2="28.65" y2="26.6" width="0" layer="19" extent="1-1"/>
+<wire x1="30.5" y1="29.6" x2="28.65" y2="26.6" width="0" layer="19" extent="1-1"/>
 </signal>
 <signal name="N$9">
 <contactref element="U5" pad="3"/>
 <contactref element="C1" pad="1"/>
-<wire x1="-7.5" y1="-3.6" x2="30.55" y2="24.2" width="0" layer="19" extent="1-1"/>
+<wire x1="28.7" y1="29.6" x2="30.55" y2="24.2" width="0" layer="19" extent="1-1"/>
 </signal>
 <signal name="VCC_REG">
@@
 <wire x1="32.2" y1="26.425" x2="32.7" y2="26.425" width="0" layer="19" extent="1-1"/>
 <wire x1="29.6" y1="26.6" x2="32.2" y2="26.425" width="0" layer="19" extent="1-1"/>
-<wire x1="-2.1" y1="-3.6" x2="29.6" y2="26.6" width="0" layer="19" extent="1-1"/>
+<wire x1="34.1" y1="29.6" x2="29.6" y2="26.6" width="0" layer="19" extent="1-1"/>
 </signal>
 <signal name="N$10">
@@
 <contactref element="U4" pad="2"/>
 <contactref element="R8" pad="2"/>
-<wire x1="-11.7" y1="-7" x2="32.7" y2="23.575" width="0" layer="19" extent="1-1"/>
+<wire x1="24.5" y1="26.2" x2="32.7" y2="23.575" width="0" layer="19" extent="1-1"/>
 </signal>
 <signal name="T~">
