File: lipolski.sch (EAGLE design)
At the start: 90 parts, among them Q1 2NMOS30V_0.1A, Q11 NMOS40V_10A, Q12 NMOS40V_10A, Q14 NMOS40V_10A, Q15 NMOS40V_10A, Q16 NMOS40V_10A, Q18 NMOS40V_10A, Q2 2PMOS50V_0.17A, Q21 PMOS30V_11A, Q22 PMOS30V_11A, Q23 NMOS40V_10A, Q24 NMOS40V_10A, Q25 PMOS30V_11A, Q26 PMOS30V_11A, Q27 NMOS40V_10A, Q28 NMOS40V_10A, Q3 2PMOS50V_0.17A, Q31 PMOS30V_11A, Q32 PMOS30V_11A, Q33 PMOS30V_11A, Q34 PMOS30V_11A, Q35 PMOS30V_11A, Q36 PMOS30V_11A, Q37 PMOS30V_11A, Q38 PMOS30V_11A, Q41 PMOS30V_11A, Q42 PMOS30V_11A, Q43 PMOS30V_11A, Q44 PMOS30V_11A, Q45 PMOS30V_11A, Q46 PMOS30V_11A, Q47 PMOS30V_11A, Q48 PMOS30V_11A, Q51 PMOS30V_11A, Q52 PMOS30V_11A, Q53 PMOS30V_11A, Q54 PMOS30V_11A, Q55 PMOS30V_11A, Q56 PMOS30V_11A, Q57 PMOS30V_11A, Q58 PMOS30V_11A, Q62 PMOS30V_11A, Q64 PMOS30V_11A, Q66 PMOS30V_11A, Q68 PMOS30V_11A, T1 TFORM_4_4311_4A4, U1 DG508BEN-T1-GE4, U10 CCR20MA_45V, U2 DG508BEN-T1-GE4, U3 74HC595, U4 LT3757IDD, U5 TC1240A

Commit message: LTC3803 simu
Changed lines of the file:
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@@
 <net name="!OE" class="0">
 <segment>
-<label x="299.72" y="175.26" size="1.778" layer="95" rot="R180" xref="yes"/>
 <pinref part="U3" gate="G$1" pin="!OE"/>
 <pinref part="R3" gate="G$1" pin="2"/>
 <wire x1="309.88" y1="175.26" x2="309.88" y2="172.72" width="0.1524" layer="91"/>
-<wire x1="309.88" y1="172.72" x2="299.72" y2="172.72" width="0.1524" layer="91"/>
-<wire x1="299.72" y1="172.72" x2="299.72" y2="175.26" width="0.1524" layer="91"/>
+<wire x1="309.88" y1="172.72" x2="297.18" y2="172.72" width="0.1524" layer="91"/>
+<wire x1="299.72" y1="175.26" x2="297.18" y2="175.26" width="0.1524" layer="91"/>
+<wire x1="297.18" y1="175.26" x2="297.18" y2="172.72" width="0.1524" layer="91"/>
+<label x="297.18" y="175.26" size="1.778" layer="95" rot="R180" xref="yes"/>
 </segment>
 </net>
