File: lipolski-control.brd (EAGLE design)
At the start: 56.2 x 21 mm, 5 parts, among them U1 ATTINYX4A8MU, U7 LTV-816S

Commit message: starting to organize board
Parts:
- added D11, D21, D31, D41, D51, D61: LEDGREEN_2V_30MA, dubec:0603+
- added U10: CCR20MA_45V, dubec:SOD-123
Connections:
- new net C1: U10.A
- new net N$16: D21.C
- new net N$17: D11.C
- new net N$18: D41.C
- new net N$2: D11.A, D21.A, D31.A, D41.A, D51.A, D61.A, U10.C
- new net N$9: D31.C
Changed lines of the file:
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@@
 <attribute name="MFG_PART_#" value="LTV-816S" x="15.24" y="10.16" size="1.778" layer="27" display="off"/>
+</element>
+<element name="D61" library="dubec" package="0603+" value="LEDGREEN_2V_30MA" x="1.7" y="-22.8">
+<attribute name="DIGIKEY_PART_#" value="160-1435-1-ND" x="1.7" y="-1.8" size="1.778" layer="27" display="off"/>
+<attribute name="LUM" value="35mcd" x="1.7" y="-1.8" size="1.778" layer="27" display="off"/>
+<attribute name="EURO" value="3.26/25" x="1.7" y="-1.8" size="1.778" layer="27" display="off"/>
+<attribute name="MANUFACTURER" value="Lite-On Inc." x="1.7" y="-1.8" size="1.778" layer="27" display="off"/>
+<attribute name="MFG_PART_#" value="LTST-C190KGKT" x="1.7" y="-1.8" size="1.778" layer="27" display="off"/>
+</element>
+<element name="D51" library="dubec" package="0603+" value="LEDGREEN_2V_30MA" x="1.7" y="-19.4">
+<attribute name="DIGIKEY_PART_#" value="160-1435-1-ND" x="1.7" y="-5.2" size="1.778" layer="27" display="off"/>
+<attribute name="LUM" value="35mcd" x="1.7" y="-5.2" size="1.778" layer="27" display="off"/>
+<attribute name="EURO" value="3.26/25" x="1.7" y="-5.2" size="1.778" layer="27" display="off"/>
+<attribute name="MANUFACTURER" value="Lite-On Inc." x="1.7" y="-5.2" size="1.778" layer="27" display="off"/>
+<attribute name="MFG_PART_#" value="LTST-C190KGKT" x="1.7" y="-5.2" size="1.778" layer="27" display="off"/>
+</element>
+<element name="D41" library="dubec" package="0603+" value="LEDGREEN_2V_30MA" x="1.7" y="-16">
+<attribute name="DIGIKEY_PART_#" value="160-1435-1-ND" x="1.7" y="-8.6" size="1.778" layer="27" display="off"/>
+<attribute name="LUM" value="35mcd" x="1.7" y="-8.6" size="1.778" layer="27" display="off"/>
+<attribute name="EURO" value="3.26/25" x="1.7" y="-8.6" size="1.778" layer="27" display="off"/>
+<attribute name="MANUFACTURER" value="Lite-On Inc." x="1.7" y="-8.6" size="1.778" layer="27" display="off"/>
+<attribute name="MFG_PART_#" value="LTST-C190KGKT" x="1.7" y="-8.6" size="1.778" layer="27" display="off"/>
+</element>
+<element name="D31" library="dubec" package="0603+" value="LEDGREEN_2V_30MA" x="1.7" y="-12.6">
+<attribute name="DIGIKEY_PART_#" value="160-1435-1-ND" x="1.7" y="-12" size="1.778" layer="27" display="off"/>
+<attribute name="LUM" value="35mcd" x="1.7" y="-12" size="1.778" layer="27" display="off"/>
+<attribute name="EURO" value="3.26/25" x="1.7" y="-12" size="1.778" layer="27" display="off"/>
+<attribute name="MANUFACTURER" value="Lite-On Inc." x="1.7" y="-12" size="1.778" layer="27" display="off"/>
+<attribute name="MFG_PART_#" value="LTST-C190KGKT" x="1.7" y="-12" size="1.778" layer="27" display="off"/>
+</element>
+<element name="D21" library="dubec" package="0603+" value="LEDGREEN_2V_30MA" x="1.7" y="-9.2">
+<attribute name="DIGIKEY_PART_#" value="160-1435-1-ND" x="1.7" y="-15.4" size="1.778" layer="27" display="off"/>
+<attribute name="LUM" value="35mcd" x="1.7" y="-15.4" size="1.778" layer="27" display="off"/>
+<attribute name="EURO" value="3.26/25" x="1.7" y="-15.4" size="1.778" layer="27" display="off"/>
+<attribute name="MANUFACTURER" value="Lite-On Inc." x="1.7" y="-15.4" size="1.778" layer="27" display="off"/>
+<attribute name="MFG_PART_#" value="LTST-C190KGKT" x="1.7" y="-15.4" size="1.778" layer="27" display="off"/>
+</element>
+<element name="D11" library="dubec" package="0603+" value="LEDGREEN_2V_30MA" x="1.7" y="-5.8">
+<attribute name="DIGIKEY_PART_#" value="160-1435-1-ND" x="1.7" y="-18.8" size="1.778" layer="27" display="off"/>
+<attribute name="LUM" value="35mcd" x="1.7" y="-18.8" size="1.778" layer="27" display="off"/>
+<attribute name="EURO" value="3.26/25" x="1.7" y="-18.8" size="1.778" layer="27" display="off"/>
+<attribute name="MANUFACTURER" value="Lite-On Inc." x="1.7" y="-18.8" size="1.778" layer="27" display="off"/>
+<attribute name="MFG_PART_#" value="LTST-C190KGKT" x="1.7" y="-18.8" size="1.778" layer="27" display="off"/>
+</element>
+<element name="U10" library="dubec" package="SOD-123" value="CCR20MA_45V" x="2.5" y="-2.1">
+<attribute name="DIGIKEY_PART_#" value="NSI45020T1GOSCT-ND" x="2.5" y="-22.5" size="1.778" layer="27" display="off"/>
+<attribute name="TOLERANCE" value="±15%" x="2.5" y="-22.5" size="1.778" layer="27" display="off"/>
+<attribute name="EURO" value="3.36/10" x="2.5" y="-22.5" size="1.778" layer="27" display="off"/>
+<attribute name="MANUFACTURER" value="ON Semiconductor" x="2.5" y="-22.5" size="1.778" layer="27" display="off"/>
+<attribute name="MFG_PART_#" value="NSI45020T1G" x="2.5" y="-22.5" size="1.778" layer="27" display="off"/>
 </element>
 </elements>
@@
 <via x="2.1" y="18.6" extent="1-16" drill="0.25"/>
 </signal>
+<signal name="C1">
+<contactref element="U10" pad="A"/>
+</signal>
+<signal name="N$2">
+<contactref element="U10" pad="C"/>
+<contactref element="D61" pad="A"/>
+<contactref element="D51" pad="A"/>
+<contactref element="D41" pad="A"/>
+<contactref element="D31" pad="A"/>
+<contactref element="D21" pad="A"/>
+<contactref element="D11" pad="A"/>
+<wire x1="0.9" y1="-19.4" x2="0.9" y2="-22.8" width="0" layer="19" extent="1-1"/>
+<wire x1="0.9" y1="-16" x2="0.9" y2="-19.4" width="0" layer="19" extent="1-1"/>
+<wire x1="0.9" y1="-12.6" x2="0.9" y2="-16" width="0" layer="19" extent="1-1"/>
+<wire x1="0.9" y1="-9.2" x2="0.9" y2="-12.6" width="0" layer="19" extent="1-1"/>
+<wire x1="0.9" y1="-5.8" x2="0.9" y2="-9.2" width="0" layer="19" extent="1-1"/>
+<wire x1="4.15" y1="-2.1" x2="0.9" y2="-5.8" width="0" layer="19" extent="1-1"/>
+</signal>
+<signal name="N$9">
+<contactref element="D31" pad="C"/>
+</signal>
+<signal name="N$16">
+<contactref element="D21" pad="C"/>
+</signal>
+<signal name="N$17">
+<contactref element="D11" pad="C"/>
+</signal>
+<signal name="N$18">
+<contactref element="D41" pad="C"/>
+</signal>
 </signals>
