File: lipolski-control.sch (EAGLE design)
At the start: 5 parts, among them U1 ATTINYX4A8MU, U7 LTV-816S

Commit message: starting to organize board
Parts:
- added D11, D21, D31, D41, D51, D61: LEDGREEN_2V_30MA, dubec:LEDGREEN_2V_30MA
- added U10: CCR20MA_45V, dubec:CCR20MA_45V
Connections:
- new net C1: U10.A
- new net N$16: D21.C
- new net N$17: D11.C
- new net N$18: D41.C
- new net N$2: D11.A, D21.A, D31.A, D41.A, D51.A, D61.A, U10.C
- new net N$9: D31.C
Changed lines of the file:
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@@
 <part name="D1" library="dubec" deviceset="D_ZENER" device="3V"/>
 <part name="U1" library="dubec" deviceset="ATTINYX4A" device="8MU"/>
+<part name="D61" library="dubec" deviceset="LED" device="GREEN_2V_30MA"/>
+<part name="D51" library="dubec" deviceset="LED" device="GREEN_2V_30MA"/>
+<part name="D41" library="dubec" deviceset="LED" device="GREEN_2V_30MA"/>
+<part name="D31" library="dubec" deviceset="LED" device="GREEN_2V_30MA"/>
+<part name="D21" library="dubec" deviceset="LED" device="GREEN_2V_30MA"/>
+<part name="D11" library="dubec" deviceset="LED" device="GREEN_2V_30MA"/>
+<part name="U10" library="dubec" deviceset="CCR" device="20MA_45V"/>
 </parts>
 <sheets>
@@
 <instance part="D1" gate="G$1" x="5.08" y="0"/>
 <instance part="U1" gate="G$1" x="-60.96" y="2.54"/>
+<instance part="D61" gate="G$1" x="-30.48" y="-38.1"/>
+<instance part="D51" gate="G$1" x="-30.48" y="-43.18"/>
+<instance part="D41" gate="G$1" x="-30.48" y="-48.26"/>
+<instance part="D31" gate="G$1" x="-30.48" y="-53.34"/>
+<instance part="D21" gate="G$1" x="-30.48" y="-58.42"/>
+<instance part="D11" gate="G$1" x="-30.48" y="-63.5"/>
+<instance part="U10" gate="G$1" x="-40.64" y="-38.1"/>
 </instances>
 <busses>
@@
 </segment>
 </net>
+<net name="C1" class="0">
+<segment>
+<pinref part="U10" gate="G$1" pin="A"/>
+<wire x1="-45.72" y1="-38.1" x2="-48.26" y2="-38.1" width="0.1524" layer="91"/>
+<label x="-48.26" y="-38.1" size="1.778" layer="95" rot="R180" xref="yes"/>
+</segment>
+</net>
+<net name="N$2" class="0">
+<segment>
+<pinref part="U10" gate="G$1" pin="C"/>
+<pinref part="D61" gate="G$1" pin="A"/>
+<wire x1="-35.56" y1="-38.1" x2="-33.02" y2="-38.1" width="0.1524" layer="91"/>
+<pinref part="D51" gate="G$1" pin="A"/>
+<wire x1="-33.02" y1="-38.1" x2="-33.02" y2="-43.18" width="0.1524" layer="91"/>
+<junction x="-33.02" y="-38.1"/>
+<pinref part="D41" gate="G$1" pin="A"/>
+<wire x1="-33.02" y1="-43.18" x2="-33.02" y2="-48.26" width="0.1524" layer="91"/>
+<junction x="-33.02" y="-43.18"/>
+<pinref part="D31" gate="G$1" pin="A"/>
+<wire x1="-33.02" y1="-48.26" x2="-33.02" y2="-53.34" width="0.1524" layer="91"/>
+<junction x="-33.02" y="-48.26"/>
+<pinref part="D21" gate="G$1" pin="A"/>
+<wire x1="-33.02" y1="-53.34" x2="-33.02" y2="-58.42" width="0.1524" layer="91"/>
+<junction x="-33.02" y="-53.34"/>
+<pinref part="D11" gate="G$1" pin="A"/>
+<wire x1="-33.02" y1="-58.42" x2="-33.02" y2="-63.5" width="0.1524" layer="91"/>
+<junction x="-33.02" y="-58.42"/>
+</segment>
+</net>
+<net name="N$9" class="0">
+<segment>
+<pinref part="D31" gate="G$1" pin="C"/>
+<wire x1="-25.4" y1="-53.34" x2="-22.86" y2="-53.34" width="0.1524" layer="91"/>
+</segment>
+</net>
+<net name="N$16" class="0">
+<segment>
+<pinref part="D21" gate="G$1" pin="C"/>
+<wire x1="-25.4" y1="-58.42" x2="-22.86" y2="-58.42" width="0.1524" layer="91"/>
+</segment>
+</net>
+<net name="N$17" class="0">
+<segment>
+<pinref part="D11" gate="G$1" pin="C"/>
+<wire x1="-25.4" y1="-63.5" x2="-22.86" y2="-63.5" width="0.1524" layer="91"/>
+</segment>
+</net>
+<net name="N$18" class="0">
+<segment>
+<pinref part="D41" gate="G$1" pin="C"/>
+<wire x1="-25.4" y1="-48.26" x2="-22.86" y2="-48.26" width="0.1524" layer="91"/>
+</segment>
+</net>
