File: lipolski-power.brd (EAGLE design)
At the start: 56.2 x 21 mm, 90 parts, among them Q1 2NMOS30V_0.1A, Q11 NMOS40V_10A, Q12 NMOS40V_10A, Q14 NMOS40V_10A, Q15 NMOS40V_10A, Q16 NMOS40V_10A, Q18 NMOS40V_10A, Q2 2PMOS50V_0.17A, Q21 PMOS30V_11A, Q22 PMOS30V_11A, Q23 NMOS40V_10A, Q24 NMOS40V_10A, Q25 PMOS30V_11A, Q26 PMOS30V_11A, Q27 NMOS40V_10A, Q28 NMOS40V_10A, Q3 2PMOS50V_0.17A, Q31 PMOS30V_11A, Q32 PMOS30V_11A, Q33 PMOS30V_11A, Q34 PMOS30V_11A, Q35 PMOS30V_11A, Q36 PMOS30V_11A, Q37 PMOS30V_11A, Q38 PMOS30V_11A, Q41 PMOS30V_11A, Q42 PMOS30V_11A, Q43 PMOS30V_11A, Q44 PMOS30V_11A, Q45 PMOS30V_11A, Q46 PMOS30V_11A, Q47 PMOS30V_11A, Q48 PMOS30V_11A, Q51 PMOS30V_11A, Q52 PMOS30V_11A, Q53 PMOS30V_11A, Q54 PMOS30V_11A, Q55 PMOS30V_11A, Q56 PMOS30V_11A, Q57 PMOS30V_11A, Q58 PMOS30V_11A, Q62 PMOS30V_11A, Q64 PMOS30V_11A, Q66 PMOS30V_11A, Q68 PMOS30V_11A, T1 TFORM_4_4311_4A4, U1 DG508BEN-T1-GE4, U10 CCR20MA_45V, U2 DG508BEN-T1-GE4, U3 74HC595, U4 LT3757IDD, U5 TC1240A

Commit message: rename
Parts:
- removed C3: CAP47NF_16V, dubec:0201P
- removed U$1: TCAP330UF_6.3V, dubec:1210+
- removed U$8: NMOS30V_30A, dubec:8-POWERWDFN
- added C6: CAP47UF_10V, dubec:0805
- added D3, D4: D_SCH20V_0.5A, dubec:SOD523+
- added Q4: 2PMOS50V_0.17A, dubec:SOT-666
- added R10: RES100K_16, dubec:0402
- added R9: RES2_10, dubec:0603
- C1: value CAP47UF_10V -> CAP4.7U_10V; device dubec:0805 -> dubec:0603
- C4: value CAP22N_50V -> CAP47N_25V
- Q1: value 2NMOS30V_0.1A -> NMOS30V_30A; device dubec:SOT-666 -> dubec:8-POWERWDFN
- Q2: value 2PMOS50V_0.17A -> 2NMOS30V_0.1A
- R5: value RES01_0.75W -> RES003_1W
- R6: value RES41.2K_16 -> RES61.9K_16
- R7: value RES6.8K_16 -> RES2.2K_16
- R8: value RES2.2K_16 -> RES15.4K_16
- U4: value LT3757IDD -> LTC3805-5IDD
- U5: value TC1240A -> LM2665M6
- moved R8 20.3 mm to (32.6, 7.80), turned to 90 degrees
- moved Q1 16.7 mm to (35.6, 8.00)
- moved U4 10.6 mm to (22.8, 26.8)
- moved Q2 7.78 mm to (42.0, 23.4)
- moved Q3 7.01 mm to (45.4, 30.4)
Connections:
- removed net FBX: R8.2, U4.2
- removed net N$1: U3.7
- new net FB: U4.3
- new net N$11: D3.A, R9.2
- new net RUN_REG: U3.7, U4.4
- net !EN_S1: now also Q2.5, R10.2; no longer Q1.5
- net BATT-: now also Q2.4, R10.1, U1.7, U1.8, U1.9; no longer Q1.4
- net C4+: now also Q4.1, Q4.4; no longer Q2.1, Q3.4
- net GS+2: now also Q3.2; no longer Q2.2
- net GS-2: now also Q3.6; no longer Q2.6
- net GS1: now also Q2.3; no longer Q1.3
- net GS6: no longer U1.7, U1.8, U1.9
- net GT+2: now also Q4.5; no longer Q3.5
- net GT-2: now also Q4.3; no longer Q3.3
- net GT1: now also Q4.6; no longer Q3.6
- net N$10: now also Q1.D; no longer U$8.D
- net N$12: now also U4.2; no longer U4.1
- net N$23: now also Q4.2; no longer Q3.2
- net N$3: now also U4.5; no longer U4.4
- net N$5: now also Q1.G, U4.6; no longer U$8.G, U4.7
- net N$6: now also R8.1, U4.9; no longer C3.2, U4.3
- net N$7: now also Q1.S, R8.2; no longer U$8.S, U4.6
- net S+: now also R9.1; no longer D2.1, D2.2, U5.1
- net S-: now also C6.1, U4.10, U4.8; no longer C3.1, R8.1, U$1.C, U4.5
- net VCC: now also C6.2, D3.C, D4.A, U5.1; no longer D2.7, D2.8, U$1.A
- net VCC_REG: now also D4.C, U4.7; no longer U4.10, U4.8, U4.9

Commit message: getting there
Parts:
- added C10: CAP47UF_10V, dubec:0805
- added C3, C8: CAP4.7U_10V, dubec:0603
- added C7: CAP4.7UF_35V, dubec:0603
- added C9: CAP22P_50V, dubec:0402
- added Q5: 2NMOS30V_0.1A, dubec:SOT-666
- added R11: RES10K_16, dubec:0402
- added R12: RES590_16, dubec:0402
- added R13: RES2.2K_16, dubec:0402
- added R14, R18: RES5.1K_16, dubec:0402
- added R15: RES100K_16, dubec:0402
- added R16: RES1.6K_16, dubec:0402
- added R17: RES402_16, dubec:0402
- added U6: AR30N60PPA-13, dubec:22-VFDFN
- added U7: LTV-816S, dubec:4-OPTO-1
- D4: value D_SCH20V_0.5A -> D_ZENER2.4V
- U5: value LM2665M6 -> TC1240A
- moved D4 44.5 mm to (-0.80, -9.00)
Connections:
- removed net FB: U4.3
- removed net T~: T1.3
- new net N$1: D4.C, R11.1, U4.3
- new net N$18: C9.1, Q5.6, R12.2
- new net N$20: C9.2, R13.1
- new net N$21: R13.2, U6.19
- new net N$22: R11.2, R16.2, U7.3
- new net N$24: R14.2, U6.1
- new net N$25: R15.2, U6.2
- new net N$26: T1.1, U6.12-17, U6.VD
- new net N$27: Q5.3, R18.2, U7.2
- new net N$29: R17.1, U7.1
- new net N$30: Q5.5, U6.3
- net BATT+: now also C7.2
- net BATT-: now also C7.1
- net N$5: now also Q5.2
- net S-: now also C8.1, D4.A, Q5.1, R16.1
- net T+: now also C10.2, R17.2, T1.3, U6.22
- net T-: now also C10.1, Q5.4, R14.1, R15.1, R18.1, U6.21, U6.5, U6.6-11, U6.GND; no longer T1.1
- net VCC: now also C3.2, C8.2; no longer D4.A
- net VCC_REG: now also C3.1, R12.1, U7.4; no longer D4.C

Commit message: .
Parts:
- removed R16: RES1.6K_16, dubec:0402
- removed U7: LTV-816S, dubec:4-OPTO-1
Connections:
- removed net N$22: R11.2, R16.2, U7.3
- removed net N$27: Q5.3, R18.2, U7.2
- removed net N$29: R17.1, U7.1
- new net FB: R11.2
- new net OPTO_A: R17.1
- new net OPTO_C: Q5.3, R18.2
- net S-: no longer R16.1
- net VCC_REG: no longer U7.4
Changed lines of the file:
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@@
 </class>
 </classes>
-<designrules name="default *">
+<designrules name="OSHPark">
 <description language="de">&lt;b&gt;EAGLE Design Rules&lt;/b&gt;
 &lt;p&gt;
@@
 <attribute name="MANUFACTURER" value="TDK Corporation" x="-5.4" y="-18.8" size="1.778" layer="27" display="off"/>
 </element>
-<element name="U7" library="dubec" package="4-OPTO-1" value="LTV-816S" x="-11.6" y="-16">
-<attribute name="TEMP" value="-50°C ~ 110°C" x="-11.6" y="-16" size="1.778" layer="27" display="off"/>
-<attribute name="DIGIKEY_PART_#" value="160-1361-5-ND" x="-11.6" y="-16" size="1.778" layer="27" display="off"/>
-<attribute name="EURO" value="5.67/25" x="-11.6" y="-16" size="1.778" layer="27" display="off"/>
-<attribute name="MFG_PART_#" value="LTV-816S" x="-11.6" y="-16" size="1.778" layer="27" display="off"/>
-<attribute name="I_FWD" value="50mA" x="-11.6" y="-16" size="1.778" layer="27" display="off"/>
-<attribute name="MANUFACTURER" value="Lite-On Inc." x="-11.6" y="-16" size="1.778" layer="27" display="off"/>
-</element>
-<element name="R16" library="dubec" package="0402" value="RES1.6K_16" x="-14.6" y="-22.4">
-<attribute name="TEMP" value="±100ppm/°C" x="-14.6" y="-22.4" size="1.778" layer="27" display="off"/>
-<attribute name="DIGIKEY_PART_#" value="541-1.60KLCT-ND" x="-14.6" y="-22.4" size="1.778" layer="27" display="off"/>
-<attribute name="TOLERANCE" value="±1%" x="-14.6" y="-22.4" size="1.778" layer="27" display="off"/>
-<attribute name="USD" value="1.82/50" x="-14.6" y="-22.4" size="1.778" layer="27" display="off"/>
-<attribute name="MFG_PART_#" value="CRCW04021K60FKED" x="-14.6" y="-22.4" size="1.778" layer="27" display="off"/>
-<attribute name="MANUFACTURER" value="Vishay Dale" x="-14.6" y="-22.4" size="1.778" layer="27" display="off"/>
-</element>
 <element name="R17" library="dubec" package="0402" value="RES402_16" x="-14.6" y="-24.6">
 <attribute name="TEMP" value="±100ppm/°C" x="-14.6" y="-24.6" size="1.778" layer="27" display="off"/>
@@
 <contactref element="C8" pad="1"/>
 <contactref element="D4" pad="A"/>
-<contactref element="R16" pad="1"/>
 <contactref element="Q5" pad="1"/>
 <wire x1="56.65" y1="27.85" x2="57.775" y2="30.4" width="0" layer="19" extent="1-1"/>
@@
 <wire x1="35.8" y1="1.85" x2="19.375" y2="3" width="0" layer="19" extent="1-1"/>
 <wire x1="-1.5" y1="-9" x2="16.1" y2="2.6" width="0" layer="19" extent="1-1"/>
-<wire x1="-15.1" y1="-22.4" x2="-1.5" y2="-9" width="0" layer="19" extent="1-1"/>
-<wire x1="-17.5" y1="-27.1" x2="-15.1" y2="-22.4" width="0" layer="19" extent="1-1"/>
+<wire x1="-17.5" y1="-27.1" x2="-1.5" y2="-9" width="0" layer="19" extent="1-1"/>
 </signal>
 <signal name="S+">
@@
 <contactref element="C3" pad="1"/>
 <contactref element="R12" pad="1"/>
-<contactref element="U7" pad="4"/>
 <wire x1="34.1" y1="29.6" x2="35.85" y2="33.2" width="0" layer="19" extent="1-1"/>
 <wire x1="29.6" y1="26.6" x2="34.1" y2="29.6" width="0" layer="19" extent="1-1"/>
 <wire x1="23.3" y1="28.225" x2="29.6" y2="26.6" width="0" layer="19" extent="1-1"/>
 <wire x1="-2.7" y1="-11.4" x2="23.3" y2="28.225" width="0" layer="19" extent="1-1"/>
-<wire x1="-12.87" y1="-11.5" x2="-2.7" y2="-11.4" width="0" layer="19" extent="1-1"/>
 </signal>
 <signal name="N$10">
@@
 <wire x1="41" y1="2.3" x2="67.005" y2="23.2" width="0" layer="19" extent="1-1"/>
 </signal>
-<signal name="N$22">
+<signal name="FB">
 <contactref element="R11" pad="2"/>
-<contactref element="U7" pad="3"/>
-<contactref element="R16" pad="2"/>
-<wire x1="-10.33" y1="-11.5" x2="-14.1" y2="-22.4" width="0" layer="19" extent="1-1"/>
-<wire x1="-1.7" y1="-7" x2="-10.33" y2="-11.5" width="0" layer="19" extent="1-1"/>
-</signal>
-<signal name="N$29">
-<contactref element="U7" pad="1"/>
+</signal>
+<signal name="OPTO_A">
 <contactref element="R17" pad="1"/>
-<wire x1="-12.87" y1="-20.5" x2="-15.1" y2="-24.6" width="0" layer="19" extent="1-1"/>
-</signal>
-<signal name="N$27">
-<contactref element="U7" pad="2"/>
+</signal>
+<signal name="OPTO_C">
 <contactref element="R18" pad="2"/>
 <contactref element="Q5" pad="3"/>
 <wire x1="-14.1" y1="-26.8" x2="-16.5" y2="-27.1" width="0" layer="19" extent="1-1"/>
-<wire x1="-10.33" y1="-20.5" x2="-14.1" y2="-26.8" width="0" layer="19" extent="1-1"/>
 </signal>
 <signal name="N$30">

Commit message: starting to organize board
Parts:
- removed C6: CAP47UF_10V, dubec:0805
- removed D11, D21, D31, D41, D51, D61: LEDGREEN_2V_30MA, dubec:0603+
- removed Q1: NMOS30V_30A, dubec:8-POWERWDFN
- removed U10: CCR20MA_45V, dubec:SOD-123
- added MVOE: NMOS30V_30A, dubec:8-POWERWDFN
- moved Q5 79.2 mm to (54.2, 8.40), turned to 180 degrees
- moved R17 77.6 mm to (58.1, 2.40)
- moved R18 76.0 mm to (52.8, 8.40), turned to 90 degrees
- moved R11 75.5 mm to (67.8, 21.2), turned to 270 degrees
- moved D4 73.0 mm to (65.7, 21.1), turned to 90 degrees
- moved C10 67.6 mm to (58.1, 4.40), turned to 270 degrees
- moved R15 65.9 mm to (58.1, 6.40), turned to 180 degrees
- moved D1 65.6 mm to (10.6, 2.70), turned to 0 degrees
- moved R14 65.4 mm to (58.1, 7.40), turned to 180 degrees
- moved R12 63.6 mm to (58.1, 8.80), turned to 180 degrees
- moved D2 62.1 mm to (11.8, 20.1)
- moved RGS1 59.8 mm to (18.6, 22.2)
- moved C9 59.7 mm to (54.4, 5.40), turned to 180 degrees
- moved R13 58.8 mm to (52.6, 5.40), turned to 180 degrees
- moved RGS4 49.9 mm to (18.8, 25.4), turned to 0 degrees
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Connections:
- removed net N$13: D41.C
- removed net N$14: D31.C
- removed net N$15: D21.C
- removed net N$16: D11.C
- removed net N$4: D11.A, D21.A, D31.A, D41.A, D51.A, D61.A, U10.C
- net C1: no longer U10.A
- net N$10: now also MVOE.D; no longer Q1.D
- net N$5: now also MVOE.G; no longer Q1.G
- net N$7: now also MVOE.S; no longer Q1.S
- net S-: no longer C6.1
- net VCC: no longer C6.2
Routing:
- net C1: track 31.2 -> 12.9 mm
- net T-: track 0.00 -> 12.5 mm
- net T+: track 0.00 -> 12.5 mm
- net S-: track 0.00 -> 12.5 mm
- net GS3: track 1.91 -> 12.0 mm, vias 2 -> 4
- net GS+2: track 1.91 -> 3.00 mm
- net GS4: track 1.91 -> 3.00 mm
- net GS5: track 1.91 -> 3.00 mm
- net C3: vias 0 -> 3
- net C2: vias 0 -> 3
- added copper zone on layer 16, net C1
- added copper zone on layer 1, net C2
- added copper zone on layer 16, net C2
- added copper zone on layer 1, net C3
