File: lipolski-power.sch (EAGLE design)
At the start: 90 parts, among them Q1 2NMOS30V_0.1A, Q11 NMOS40V_10A, Q12 NMOS40V_10A, Q14 NMOS40V_10A, Q15 NMOS40V_10A, Q16 NMOS40V_10A, Q18 NMOS40V_10A, Q2 2PMOS50V_0.17A, Q21 PMOS30V_11A, Q22 PMOS30V_11A, Q23 NMOS40V_10A, Q24 NMOS40V_10A, Q25 PMOS30V_11A, Q26 PMOS30V_11A, Q27 NMOS40V_10A, Q28 NMOS40V_10A, Q3 2PMOS50V_0.17A, Q31 PMOS30V_11A, Q32 PMOS30V_11A, Q33 PMOS30V_11A, Q34 PMOS30V_11A, Q35 PMOS30V_11A, Q36 PMOS30V_11A, Q37 PMOS30V_11A, Q38 PMOS30V_11A, Q41 PMOS30V_11A, Q42 PMOS30V_11A, Q43 PMOS30V_11A, Q44 PMOS30V_11A, Q45 PMOS30V_11A, Q46 PMOS30V_11A, Q47 PMOS30V_11A, Q48 PMOS30V_11A, Q51 PMOS30V_11A, Q52 PMOS30V_11A, Q53 PMOS30V_11A, Q54 PMOS30V_11A, Q55 PMOS30V_11A, Q56 PMOS30V_11A, Q57 PMOS30V_11A, Q58 PMOS30V_11A, Q62 PMOS30V_11A, Q64 PMOS30V_11A, Q66 PMOS30V_11A, Q68 PMOS30V_11A, T1 TFORM_4_4311_4A4, U1 DG508BEN-T1-GE4, U10 CCR20MA_45V, U2 DG508BEN-T1-GE4, U3 74HC595, U4 LT3757IDD, U5 TC1240A

Commit message: rename
Parts:
- removed C3: CAP47NF_16V, dubec:CAP47NF_16V
- removed U$1: TCAP330UF_6.3V, dubec:TCAP330UF_6.3V
- removed U$8: NMOS30V_30A, dubec:NMOS30V_30A
- added C6: CAP47UF_10V, dubec:CAP47UF_10V
- added D3, D4: D_SCH20V_0.5A, dubec:D_SCH20V_0.5A
- added Q4: 2PMOS50V_0.17A, dubec:2PMOS50V_0.17A
- added R10: RES100K_16, dubec:RES100K_16
- added R9: RES2_10, dubec:RES2_10
- C1: value CAP47UF_10V -> CAP4.7U_10V; device dubec:CAP47UF_10V -> dubec:CAP4.7U_10V
- C4: value CAP22N_50V -> CAP47N_25V; device dubec:CAP22N_50V -> dubec:CAP47N_25V
- Q1: value 2NMOS30V_0.1A -> NMOS30V_30A; device dubec:2NMOS30V_0.1A -> dubec:NMOS30V_30A
- Q2: value 2PMOS50V_0.17A -> 2NMOS30V_0.1A; device dubec:2PMOS50V_0.17A -> dubec:2NMOS30V_0.1A
- R5: value RES01_0.75W -> RES003_1W; device dubec:RES01_0.75W -> dubec:RES003_1W
- R6: value RES41.2K_16 -> RES61.9K_16; device dubec:RES41.2K_16 -> dubec:RES61.9K_16
- R7: value RES6.8K_16 -> RES2.2K_16; device dubec:RES6.8K_16 -> dubec:RES2.2K_16
- R8: value RES2.2K_16 -> RES15.4K_16; device dubec:RES2.2K_16 -> dubec:RES15.4K_16
- U4: value LT3757IDD -> LTC3805-5IDD; device dubec:LT3757IDD -> dubec:LTC3805-5IDD
- U5: value TC1240A -> LM2665M6; device dubec:TC1240A -> dubec:LM2665M6
Connections:
- removed net FBX: R8.2, U4.FBX
- removed net N$1: U3.Q7
- new net FB: U4.FB
- new net N$11: D3.A, R9.2
- new net RUN_REG: U3.Q7, U4.RUN
- net !EN_S1: now also Q2G$2.G, R10.2; no longer Q1G$2.G
- net BATT-: now also Q2G$2.S, R10.1, U1.S6, U1.S7, U1.S8; no longer Q1G$2.S
- net C4+: now also Q4G$1.S, Q4G$2.S; no longer Q2G$1.S, Q3G$2.S
- net GS+2: now also Q3G$1.G; no longer Q2G$1.G
- net GS-2: now also Q3G$1.D; no longer Q2G$1.D
- net GS1: now also Q2G$2.D; no longer Q1G$2.D
- net GS6: no longer U1.S6, U1.S7, U1.S8
- net GT+2: now also Q4G$2.G; no longer Q3G$2.G
- net GT-2: now also Q4G$2.D; no longer Q3G$2.D
- net GT1: now also Q4G$1.D; no longer Q3G$1.D
- net N$10: now also Q1.D; no longer U$8.D
- net N$12: now also U4.I_TH; no longer U4.VC
- net N$23: now also Q4G$1.G; no longer Q3G$1.G
- net N$3: now also U4.FS; no longer U4.RT
- net N$5: now also Q1.G; no longer U$8.G
- net N$6: now also R8.1, U4.I_SENSE; no longer C3.2, U4.SS
- net N$7: now also Q1.S, R8.2; no longer U$8.S, U4.SENSE
- net S+: now also R9.1; no longer D2G$1.A, D2G$2.A, U5.VIN
- net S-: now also C6.1, U4.OC, U5.SD; no longer C3.1, R8.1, U$1.C, U5.SHDN
- net VCC: now also C6.2, D3.C, D4.A, U5.VIN; no longer D2G$1.C, D2G$2.C, U$1.A
- net VCC_REG: now also D4.C, U4.VCC, U5.OUT; no longer U4.!SHDN, U4.INTVCC, U4.VIN, U5.VOUT
Other:
- moved on the sheet: C1, C2, C4, C5, D11, D21, D31, D41, D51, D61, Q3G$1, R3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

Commit message: getting there
Parts:
- added C10: CAP47UF_10V, dubec:CAP47UF_10V
- added C3, C8: CAP4.7U_10V, dubec:CAP4.7U_10V
- added C7: CAP4.7UF_35V, dubec:CAP4.7UF_35V
- added C9: CAP22P_50V, dubec:CAP22P_50V
- added Q5: 2NMOS30V_0.1A, dubec:2NMOS30V_0.1A
- added R11: RES10K_16, dubec:RES10K_16
- added R12: RES590_16, dubec:RES590_16
- added R13: RES2.2K_16, dubec:RES2.2K_16
- added R14, R18: RES5.1K_16, dubec:RES5.1K_16
- added R15: RES100K_16, dubec:RES100K_16
- added R16: RES1.6K_16, dubec:RES1.6K_16
- added R17: RES402_16, dubec:RES402_16
- added U6: AR30N60PPA-13, dubec:AR30N60PPA-13
- added U7: LTV-816S, dubec:LTV-816S
- D4: value D_SCH20V_0.5A -> D_ZENER2.4V; device dubec:D_SCH20V_0.5A -> dubec:D_ZENER2.4V
- U5: value LM2665M6 -> TC1240A; device dubec:LM2665M6 -> dubec:TC1240A
Connections:
- removed net FB: U4.FB
- removed net T~: T1.2
- new net N$1: D4.C, R11.1, U4.FB
- new net N$18: C9.1, Q5G$1.D, R12.2
- new net N$20: C9.2, R13.1
- new net N$21: R13.2, U6.SYNC
- new net N$22: R11.2, R16.2, U7.E
- new net N$24: R14.2, U6.TON
- new net N$25: R15.2, U6.TOFF/EN
- new net N$26: T1.1, U6.VD
- new net N$27: Q5G$2.D, R18.2, U7.K
- new net N$29: R17.1, U7.A
- new net N$30: Q5G$2.G, U6.SFB
- net BATT+: now also C7.2
- net BATT-: now also C7.1
- net N$5: now also Q5G$1.G
- net S-: now also C8.1, D4.A, Q5G$1.S, R16.1, U5.SHDN; no longer U5.SD
- net T+: now also C10.2, R17.2, T1.2, U6.VCC
- net T-: now also C10.1, Q5G$2.S, R14.1, R15.1, R18.1, U6.GND, U6.VS; no longer T1.1
- net VCC: now also C3.2, C8.2; no longer D4.A
- net VCC_REG: now also C3.1, R12.1, U5.VOUT, U7.C; no longer D4.C, U5.OUT
Other:
- note added: "Charge IN"
- note added: "Charge OUT"
- moved on the sheet: C1, C2, C4, C5, C6, D11, D1G$1, D1G$2, D1G$3, D1G$4, D21, D2G$3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

Commit message: .
Parts:
- removed R16: RES1.6K_16, dubec:RES1.6K_16
- removed U7: LTV-816S, dubec:LTV-816S
Connections:
- removed net N$22: R11.2, R16.2, U7.E
- removed net N$27: Q5G$2.D, R18.2, U7.K
- removed net N$29: R17.1, U7.A
- new net FB: R11.2
- new net OPTO_A: R17.1
- new net OPTO_C: Q5G$2.D, R18.2
- net S-: no longer R16.1
- net VCC_REG: no longer U7.C
Other:
- note added: "Electric Potential Hell"
- note added: "OPTO"
- note added: "Repetitive Strain Injury"
- note removed: "Pick-N-Place Hell"
- note removed: "Reception of the Electric Potential Hell"
- moved on the sheet: C9, R12, R17
Changed lines of the file:
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@@
 <part name="R15" library="dubec" deviceset="RES" device="100K_16"/>
 <part name="C10" library="dubec" deviceset="CAP" device="47UF_10V"/>
-<part name="U7" library="dubec" deviceset="LTV-8" device="16S"/>
-<part name="R16" library="dubec" deviceset="RES" device="1.6K_16"/>
 <part name="R17" library="dubec" deviceset="RES" device="402_16"/>
 <part name="R18" library="dubec" deviceset="RES" device="5.1K_16"/>
@@
 <wire x1="5.08" y1="5.08" x2="5.08" y2="101.6" width="0.1524" layer="94"/>
 <wire x1="307.34" y1="101.6" x2="307.34" y2="5.08" width="0.1524" layer="94"/>
-<text x="-127" y="60.96" size="3.81" layer="94">Pick-N-Place Hell</text>
+<text x="-127" y="60.96" size="3.81" layer="94">Repetitive Strain Injury</text>
 <wire x1="60.96" y1="86.36" x2="60.96" y2="10.16" width="0.1524" layer="94" style="shortdash"/>
-<text x="12.7" y="91.44" size="3.81" layer="94">Reception of the Electric Potential Hell</text>
+<text x="12.7" y="91.44" size="3.81" layer="94">Electric Potential Hell</text>
 <wire x1="5.08" y1="-5.08" x2="223.52" y2="-5.08" width="0.1524" layer="94"/>
 <wire x1="5.08" y1="-91.44" x2="5.08" y2="-5.08" width="0.1524" layer="94"/>
@@
 <text x="139.7" y="-12.7" size="3.81" layer="94">Charge OUT</text>
 <text x="129.54" y="-12.7" size="3.81" layer="94" align="bottom-right">Charge IN</text>
+<wire x1="129.54" y1="-55.88" x2="139.7" y2="-55.88" width="0.1524" layer="94"/>
+<wire x1="139.7" y1="-55.88" x2="139.7" y2="-66.04" width="0.1524" layer="94"/>
+<wire x1="139.7" y1="-66.04" x2="129.54" y2="-66.04" width="0.1524" layer="94"/>
+<wire x1="129.54" y1="-66.04" x2="129.54" y2="-55.88" width="0.1524" layer="94"/>
+<text x="134.62" y="-60.96" size="1.778" layer="94" align="bottom-center">OPTO</text>
 </plain>
 <instances>
@@
 <instance part="R11" gate="G$1" x="109.22" y="-63.5"/>
 <instance part="D4" gate="G$1" x="99.06" y="-68.58" rot="R90"/>
-<instance part="R12" gate="G$1" x="119.38" y="-45.72" rot="R270"/>
-<instance part="C9" gate="G$1" x="133.35" y="-50.8"/>
+<instance part="R12" gate="G$1" x="119.38" y="-43.18" rot="R270"/>
+<instance part="C9" gate="G$1" x="133.35" y="-48.26"/>
 <instance part="R13" gate="G$1" x="167.64" y="-50.8"/>
 <instance part="R14" gate="G$1" x="167.64" y="-40.64"/>
@@
 <instance part="C10" gate="G$1" x="160.02" y="-33.02" rot="R90"/>
 <instance part="Q2" gate="G$1" x="129.54" y="15.24" rot="MR270"/>
-<instance part="U7" gate="G$1" x="134.62" y="-60.96" rot="MR0"/>
-<instance part="R16" gate="G$1" x="114.3" y="-68.58" rot="R90"/>
-<instance part="R17" gate="G$1" x="144.78" y="-45.72" rot="R90"/>
+<instance part="R17" gate="G$1" x="144.78" y="-43.18" rot="R90"/>
 <instance part="R18" gate="G$1" x="152.4" y="-63.5" rot="R180"/>
 <instance part="Q5" gate="G$1" x="119.38" y="-55.88"/>
@@
 <junction x="93.98" y="-78.74"/>
 <junction x="104.14" y="-78.74"/>
-<wire x1="119.38" y1="-78.74" x2="114.3" y2="-78.74" width="0.1524" layer="91"/>
-<wire x1="114.3" y1="-78.74" x2="104.14" y2="-78.74" width="0.1524" layer="91"/>
+<wire x1="119.38" y1="-78.74" x2="104.14" y2="-78.74" width="0.1524" layer="91"/>
 <wire x1="99.06" y1="-71.12" x2="99.06" y2="-78.74" width="0.1524" layer="91"/>
 <junction x="99.06" y="-78.74"/>
 <pinref part="D4" gate="G$1" pin="A"/>
-<pinref part="R16" gate="G$1" pin="1"/>
 <pinref part="Q5" gate="G$1" pin="S"/>
 <wire x1="119.38" y1="-60.96" x2="119.38" y2="-78.74" width="0.1524" layer="91"/>
-<wire x1="114.3" y1="-71.12" x2="114.3" y2="-78.74" width="0.1524" layer="91"/>
-<junction x="114.3" y="-78.74"/>
 </segment>
 <segment>
@@
 <junction x="160.02" y="-25.4"/>
 <pinref part="R17" gate="G$1" pin="2"/>
-<wire x1="144.78" y1="-25.4" x2="144.78" y2="-43.18" width="0.1524" layer="91"/>
+<wire x1="144.78" y1="-25.4" x2="144.78" y2="-40.64" width="0.1524" layer="91"/>
 <junction x="144.78" y="-25.4"/>
 </segment>
@@
 <junction x="76.2" y="-38.1"/>
 <pinref part="R12" gate="G$1" pin="1"/>
-<pinref part="U7" gate="G$1" pin="C"/>
-<wire x1="124.46" y1="-58.42" x2="127" y2="-58.42" width="0.1524" layer="91"/>
-<wire x1="124.46" y1="-38.1" x2="124.46" y2="-58.42" width="0.1524" layer="91"/>
 <wire x1="76.2" y1="-38.1" x2="119.38" y2="-38.1" width="0.1524" layer="91"/>
-<wire x1="119.38" y1="-38.1" x2="124.46" y2="-38.1" width="0.1524" layer="91"/>
-<wire x1="119.38" y1="-38.1" x2="119.38" y2="-43.18" width="0.1524" layer="91"/>
-<junction x="119.38" y="-38.1"/>
+<wire x1="119.38" y1="-38.1" x2="119.38" y2="-40.64" width="0.1524" layer="91"/>
 </segment>
 </net>
@@
 <wire x1="96.52" y1="-48.26" x2="99.06" y2="-48.26" width="0.1524" layer="91"/>
 <wire x1="96.52" y1="-48.26" x2="96.52" y2="-53.34" width="0.1524" layer="91"/>
-<wire x1="96.52" y1="-53.34" x2="111.76" y2="-53.34" width="0.1524" layer="91"/>
-<wire x1="111.76" y1="-53.34" x2="111.76" y2="-58.42" width="0.1524" layer="91"/>
+<wire x1="96.52" y1="-53.34" x2="109.22" y2="-53.34" width="0.1524" layer="91"/>
+<wire x1="109.22" y1="-53.34" x2="109.22" y2="-58.42" width="0.1524" layer="91"/>
 <junction x="96.52" y="-48.26"/>
 <pinref part="Q5" gate="G$1" pin="G"/>
-<wire x1="111.76" y1="-58.42" x2="114.3" y2="-58.42" width="0.1524" layer="91"/>
+<wire x1="109.22" y1="-58.42" x2="114.3" y2="-58.42" width="0.1524" layer="91"/>
 </segment>
 </net>
@@
 <segment>
 <pinref part="R12" gate="G$1" pin="2"/>
+<wire x1="119.38" y1="-45.72" x2="119.38" y2="-48.26" width="0.1524" layer="91"/>
+<pinref part="C9" gate="G$1" pin="1"/>
 <wire x1="119.38" y1="-48.26" x2="119.38" y2="-50.8" width="0.1524" layer="91"/>
-<pinref part="C9" gate="G$1" pin="1"/>
-<wire x1="119.38" y1="-50.8" x2="130.81" y2="-50.8" width="0.1524" layer="91"/>
 <pinref part="Q5" gate="G$1" pin="D"/>
-<junction x="119.38" y="-50.8"/>
+<wire x1="119.38" y1="-48.26" x2="130.81" y2="-48.26" width="0.1524" layer="91"/>
+<junction x="119.38" y="-48.26"/>
 </segment>
 </net>
@@
 <pinref part="C9" gate="G$1" pin="2"/>
 <pinref part="R13" gate="G$1" pin="1"/>
-<wire x1="138.43" y1="-50.8" x2="165.1" y2="-50.8" width="0.1524" layer="91"/>
+<wire x1="138.43" y1="-48.26" x2="152.4" y2="-48.26" width="0.1524" layer="91"/>
+<wire x1="152.4" y1="-48.26" x2="152.4" y2="-50.8" width="0.1524" layer="91"/>
+<wire x1="152.4" y1="-50.8" x2="165.1" y2="-50.8" width="0.1524" layer="91"/>
 </segment>
 </net>
@@
 </segment>
 </net>
-<net name="N$22" class="0">
+<net name="FB" class="0">
 <segment>
 <pinref part="R11" gate="G$1" pin="2"/>
-<pinref part="U7" gate="G$1" pin="E"/>
-<wire x1="111.76" y1="-63.5" x2="114.3" y2="-63.5" width="0.1524" layer="91"/>
-<pinref part="R16" gate="G$1" pin="2"/>
-<wire x1="114.3" y1="-63.5" x2="127" y2="-63.5" width="0.1524" layer="91"/>
-<wire x1="114.3" y1="-63.5" x2="114.3" y2="-66.04" width="0.1524" layer="91"/>
-<junction x="114.3" y="-63.5"/>
-</segment>
-</net>
-<net name="N$29" class="0">
-<segment>
-<pinref part="U7" gate="G$1" pin="A"/>
-<wire x1="144.78" y1="-58.42" x2="142.24" y2="-58.42" width="0.1524" layer="91"/>
+<wire x1="111.76" y1="-63.5" x2="129.54" y2="-63.5" width="0.1524" layer="91"/>
+<label x="129.54" y="-63.5" size="1.778" layer="95" rot="R270" xref="yes"/>
+</segment>
+</net>
+<net name="OPTO_A" class="0">
+<segment>
 <pinref part="R17" gate="G$1" pin="1"/>
-<wire x1="144.78" y1="-48.26" x2="144.78" y2="-58.42" width="0.1524" layer="91"/>
-</segment>
-</net>
-<net name="N$27" class="0">
-<segment>
-<pinref part="U7" gate="G$1" pin="K"/>
+<wire x1="144.78" y1="-45.72" x2="144.78" y2="-58.42" width="0.1524" layer="91"/>
+<wire x1="144.78" y1="-58.42" x2="139.7" y2="-58.42" width="0.1524" layer="91"/>
+<label x="139.7" y="-58.42" size="1.778" layer="95" rot="R90" xref="yes"/>
+</segment>
+</net>
+<net name="OPTO_C" class="0">
+<segment>
 <pinref part="R18" gate="G$1" pin="2"/>
-<wire x1="142.24" y1="-63.5" x2="144.78" y2="-63.5" width="0.1524" layer="91"/>
+<wire x1="139.7" y1="-63.5" x2="144.78" y2="-63.5" width="0.1524" layer="91"/>
 <wire x1="144.78" y1="-63.5" x2="149.86" y2="-63.5" width="0.1524" layer="91"/>
 <wire x1="144.78" y1="-63.5" x2="144.78" y2="-68.58" width="0.1524" layer="91"/>
@@
 <pinref part="Q5" gate="G$2" pin="D"/>
 <wire x1="144.78" y1="-68.58" x2="147.32" y2="-68.58" width="0.1524" layer="91"/>
-</segment>
-</net>
+<label x="139.7" y="-63.5" size="1.778" layer="95" rot="R270" xref="yes"/>
+</segment>
+</net>

Commit message: starting to organize board
Parts:
- removed C6: CAP47UF_10V, dubec:CAP47UF_10V
- removed D11, D21, D31, D41, D51, D61: LEDGREEN_2V_30MA, dubec:LEDGREEN_2V_30MA
- removed U10: CCR20MA_45V, dubec:CCR20MA_45V
- renumbered Q1 to MVOE
Connections:
- removed net N$13: D41.C
- removed net N$14: D31.C
- removed net N$15: D21.C
- removed net N$16: D11.C
- removed net N$4: D11.A, D21.A, D31.A, D41.A, D51.A, D61.A, U10.C
- net C1: no longer U10.A
- net S-: no longer C6.1
- net VCC: no longer C6.2
Other:
- moved on the sheet: C7, C8, D1G$1, D1G$2, D1G$3, D1G$4, D2G$3, D2G$4, D3, Q2G$1, Q2G$2, Q3G$1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
