File: lipovsky-power.sch (EAGLE design)
At the start: 99 parts, among them Q11 NMOS40V_10A, Q12 NMOS40V_10A, Q14 NMOS40V_10A, Q15 NMOS40V_10A, Q16 NMOS40V_10A, Q18 NMOS40V_10A, Q2 2NMOS30V_0.1A, Q21 PMOS30V_11A, Q22 PMOS30V_11A, Q23 NMOS40V_10A, Q24 NMOS40V_10A, Q25 PMOS30V_11A, Q26 PMOS30V_11A, Q27 NMOS40V_10A, Q28 NMOS40V_10A, Q3 2PMOS50V_0.17A, Q31 PMOS30V_11A, Q32 PMOS30V_11A, Q33 PMOS30V_11A, Q34 PMOS30V_11A, Q35 PMOS30V_11A, Q36 PMOS30V_11A, Q37 PMOS30V_11A, Q38 PMOS30V_11A, Q4 2PMOS50V_0.17A, Q41 PMOS30V_11A, Q42 PMOS30V_11A, Q43 PMOS30V_11A, Q44 PMOS30V_11A, Q45 PMOS30V_11A, Q46 PMOS30V_11A, Q47 PMOS30V_11A, Q48 PMOS30V_11A, Q5 2NMOS30V_0.1A, Q51 PMOS30V_11A, Q52 PMOS30V_11A, Q53 PMOS30V_11A, Q54 PMOS30V_11A, Q55 PMOS30V_11A, Q56 PMOS30V_11A, Q57 PMOS30V_11A, Q58 PMOS30V_11A, Q62 PMOS30V_11A, Q64 PMOS30V_11A, Q66 PMOS30V_11A, Q68 PMOS30V_11A, T1 TFORM_4_4311_4A4, U1 DG508BEN-T1-GE4, U2 DG508BEN-T1-GE4, U3 74HC595, U4 LTC3805-5IDD, U5 TC1240A, U6 AR30N60PPA-13

Commit message: Getting there
Parts:
- renumbered MVOE to Q1
Other:
- moved on the sheet: C2, C3
Changed lines of the file:
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@@
 <part name="R3" library="dubec" deviceset="RES" device="4.7K_16" value="RES4.7K_16"/>
 <part name="R4" library="dubec" deviceset="RES" device="4.7K_16" value="RES4.7K_16"/>
-<part name="MVOE" library="dubec" deviceset="NMOS" device="30V_30A"/>
+<part name="Q1" library="dubec" deviceset="NMOS" device="30V_30A"/>
 <part name="R5" library="dubec" deviceset="RES" device="003_1W" value="RES003_1W"/>
 <part name="U1" library="dubec" deviceset="DG508B" device="EN-T1-GE4"/>
@@
 <instance part="R3" gate="G$1" x="254" y="38.1" rot="R180"/>
 <instance part="R4" gate="G$1" x="251.46" y="53.34"/>
-<instance part="MVOE" gate="G$1" x="104.14" y="-45.72"/>
+<instance part="Q1" gate="G$1" x="104.14" y="-45.72"/>
 <instance part="R5" gate="G$1" x="104.14" y="-68.58" rot="R90"/>
 <instance part="U1" gate="G$1" x="111.76" y="63.5" rot="R180"/>
@@
 <instance part="R7" gate="G$1" x="55.88" y="-66.04"/>
 <instance part="C4" gate="G$1" x="50.8" y="-73.66" rot="R90"/>
-<instance part="C2" gate="G$1" x="50.8" y="-45.72" rot="R90"/>
+<instance part="C2" gate="G$1" x="48.26" y="-45.72" rot="R90"/>
 <instance part="C1" gate="G$1" x="15.24" y="-38.1" rot="R90"/>
 <instance part="C5" gate="G$1" x="73.66" y="-27.94" rot="R90"/>
@@
 <instance part="D3" gate="G$1" x="30.48" y="25.4"/>
 <instance part="R10" gate="G$1" x="116.84" y="22.86" rot="R90"/>
-<instance part="C3" gate="G$1" x="43.18" y="-27.94" rot="R90"/>
+<instance part="C3" gate="G$1" x="45.72" y="-27.94" rot="R90"/>
 <instance part="C7" gate="G$1" x="43.18" y="55.88" rot="R90"/>
 <instance part="C8" gate="G$1" x="261.62" y="76.2"/>
@@
 <pinref part="U5" gate="G$1" pin="GND"/>
 <wire x1="30.48" y1="-48.26" x2="30.48" y2="-50.8" width="0.1524" layer="91"/>
-<wire x1="30.48" y1="-50.8" x2="40.64" y2="-50.8" width="0.1524" layer="91"/>
+<wire x1="30.48" y1="-50.8" x2="43.18" y2="-50.8" width="0.1524" layer="91"/>
 <pinref part="U5" gate="G$1" pin="SHDN"/>
 <pinref part="C5" gate="G$1" pin="1"/>
 <wire x1="73.66" y1="-30.48" x2="73.66" y2="-33.02" width="0.1524" layer="91"/>
-<wire x1="73.66" y1="-33.02" x2="40.64" y2="-33.02" width="0.1524" layer="91"/>
-<wire x1="40.64" y1="-33.02" x2="40.64" y2="-50.8" width="0.1524" layer="91"/>
-<junction x="40.64" y="-33.02"/>
-<label x="30.48" y="-53.34" size="1.778" layer="95" rot="R270" xref="yes"/>
-<wire x1="30.48" y1="-50.8" x2="30.48" y2="-53.34" width="0.1524" layer="91"/>
-<junction x="30.48" y="-50.8"/>
+<wire x1="73.66" y1="-33.02" x2="43.18" y2="-33.02" width="0.1524" layer="91"/>
+<wire x1="43.18" y1="-33.02" x2="40.64" y2="-33.02" width="0.1524" layer="91"/>
+<label x="76.2" y="-81.28" size="1.778" layer="95" rot="R270" xref="yes"/>
 <pinref part="C2" gate="G$1" pin="1"/>
 <pinref part="R6" gate="G$1" pin="1"/>
@@
 <junction x="45.72" y="-60.96"/>
 <pinref part="U4" gate="G$1" pin="SYNC"/>
-<wire x1="60.96" y1="-50.8" x2="50.8" y2="-50.8" width="0.1524" layer="91"/>
-<wire x1="50.8" y1="-50.8" x2="45.72" y2="-50.8" width="0.1524" layer="91"/>
-<wire x1="50.8" y1="-48.26" x2="50.8" y2="-50.8" width="0.1524" layer="91"/>
-<junction x="50.8" y="-50.8"/>
+<wire x1="60.96" y1="-50.8" x2="48.26" y2="-50.8" width="0.1524" layer="91"/>
+<wire x1="48.26" y1="-50.8" x2="45.72" y2="-50.8" width="0.1524" layer="91"/>
+<wire x1="48.26" y1="-48.26" x2="48.26" y2="-50.8" width="0.1524" layer="91"/>
+<junction x="48.26" y="-50.8"/>
 <pinref part="R5" gate="G$1" pin="1"/>
 <wire x1="104.14" y1="-71.12" x2="104.14" y2="-78.74" width="0.1524" layer="91"/>
@@
 <pinref part="U4" gate="G$1" pin="GND"/>
 <wire x1="76.2" y1="-78.74" x2="76.2" y2="-71.12" width="0.1524" layer="91"/>
-<wire x1="40.64" y1="-50.8" x2="45.72" y2="-50.8" width="0.1524" layer="91"/>
-<junction x="40.64" y="-50.8"/>
 <junction x="45.72" y="-50.8"/>
+<wire x1="43.18" y1="-50.8" x2="45.72" y2="-50.8" width="0.1524" layer="91"/>
 <wire x1="104.14" y1="-78.74" x2="119.38" y2="-78.74" width="0.1524" layer="91"/>
 <junction x="104.14" y="-78.74"/>
 <pinref part="Q5" gate="G$1" pin="S"/>
 <wire x1="119.38" y1="-78.74" x2="119.38" y2="-60.96" width="0.1524" layer="91"/>
+<wire x1="43.18" y1="-33.02" x2="43.18" y2="-50.8" width="0.1524" layer="91"/>
+<junction x="43.18" y="-33.02"/>
+<junction x="43.18" y="-50.8"/>
+<wire x1="76.2" y1="-78.74" x2="76.2" y2="-81.28" width="0.1524" layer="91"/>
 </segment>
 </net>
@@
 <wire x1="30.48" y1="-22.86" x2="30.48" y2="-20.32" width="0.1524" layer="91"/>
 <wire x1="30.48" y1="-20.32" x2="25.4" y2="-20.32" width="0.1524" layer="91"/>
-<wire x1="30.48" y1="-20.32" x2="43.18" y2="-20.32" width="0.1524" layer="91"/>
-<wire x1="43.18" y1="-20.32" x2="43.18" y2="-22.86" width="0.1524" layer="91"/>
+<wire x1="30.48" y1="-20.32" x2="45.72" y2="-20.32" width="0.1524" layer="91"/>
+<wire x1="45.72" y1="-20.32" x2="45.72" y2="-22.86" width="0.1524" layer="91"/>
 <junction x="30.48" y="-20.32"/>
 <label x="25.4" y="-20.32" size="1.778" layer="95" rot="R180" xref="yes"/>
@@
 <segment>
 <pinref part="U5" gate="G$1" pin="VOUT"/>
-<wire x1="40.64" y1="-38.1" x2="43.18" y2="-38.1" width="0.1524" layer="91"/>
-<wire x1="43.18" y1="-38.1" x2="50.8" y2="-38.1" width="0.1524" layer="91"/>
-<wire x1="50.8" y1="-38.1" x2="76.2" y2="-38.1" width="0.1524" layer="91"/>
+<wire x1="40.64" y1="-38.1" x2="45.72" y2="-38.1" width="0.1524" layer="91"/>
+<wire x1="45.72" y1="-38.1" x2="48.26" y2="-38.1" width="0.1524" layer="91"/>
+<wire x1="48.26" y1="-38.1" x2="76.2" y2="-38.1" width="0.1524" layer="91"/>
 <wire x1="76.2" y1="-38.1" x2="76.2" y2="-40.64" width="0.1524" layer="91"/>
-<junction x="43.18" y="-38.1"/>
+<junction x="45.72" y="-38.1"/>
 <pinref part="C2" gate="G$1" pin="2"/>
 <pinref part="U4" gate="G$1" pin="VCC"/>
 <pinref part="C3" gate="G$1" pin="1"/>
-<wire x1="43.18" y1="-30.48" x2="43.18" y2="-38.1" width="0.1524" layer="91"/>
+<wire x1="45.72" y1="-30.48" x2="45.72" y2="-38.1" width="0.1524" layer="91"/>
 <junction x="76.2" y="-38.1"/>
 <pinref part="R12" gate="G$1" pin="1"/>
 <wire x1="76.2" y1="-38.1" x2="119.38" y2="-38.1" width="0.1524" layer="91"/>
 <wire x1="119.38" y1="-38.1" x2="119.38" y2="-40.64" width="0.1524" layer="91"/>
-<wire x1="50.8" y1="-38.1" x2="50.8" y2="-40.64" width="0.1524" layer="91"/>
-<junction x="50.8" y="-38.1"/>
+<wire x1="48.26" y1="-38.1" x2="48.26" y2="-40.64" width="0.1524" layer="91"/>
+<junction x="48.26" y="-38.1"/>
 </segment>
 </net>
@@
 <wire x1="124.46" y1="-33.02" x2="104.14" y2="-33.02" width="0.1524" layer="91"/>
 <wire x1="104.14" y1="-33.02" x2="104.14" y2="-40.64" width="0.1524" layer="91"/>
-<pinref part="MVOE" gate="G$1" pin="D"/>
+<pinref part="Q1" gate="G$1" pin="D"/>
 <wire x1="124.46" y1="-25.4" x2="124.46" y2="-33.02" width="0.1524" layer="91"/>
 <junction x="124.46" y="-33.02"/>
@@
 <net name="SENSE" class="0">
 <segment>
-<pinref part="MVOE" gate="G$1" pin="S"/>
+<pinref part="Q1" gate="G$1" pin="S"/>
 <pinref part="R5" gate="G$1" pin="2"/>
 <wire x1="104.14" y1="-50.8" x2="104.14" y2="-58.42" width="0.1524" layer="91"/>
@@
 <segment>
 <pinref part="U4" gate="G$1" pin="GATE"/>
-<pinref part="MVOE" gate="G$1" pin="G"/>
+<pinref part="Q1" gate="G$1" pin="G"/>
 <wire x1="91.44" y1="-48.26" x2="96.52" y2="-48.26" width="0.1524" layer="91"/>
 <wire x1="96.52" y1="-48.26" x2="99.06" y2="-48.26" width="0.1524" layer="91"/>

Commit message: connectors
Parts:
- added J1, J2, J3, J4: M04-929J, dubec:M04-929J
Connections:
- removed net N$19: U3.Q7S
- removed net N$30: Q5G$2.G, U6.SFB
- new net Q7S: J1.4, U3.Q7S
- new net SFB: J1.3, Q5G$2.G, U6.SFB
- net !OE: now also J3.2
- net BATT-: now also J1.2
- net CP: now also J3.3
- net DS: now also J3.4
- net FB: now also J2.4
- net OPTO_A: now also J2.2
- net OPTO_C: now also J2.3
- net S+: now also J4.2
- net S-: now also J1.1, J2.1, J3.1, J4.1
- net VCC: now also J4.3
- net VCC_REG: now also J4.4
Changed lines of the file:
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@@
 <part name="R18" library="dubec" deviceset="RES" device="5.1K_16"/>
 <part name="Q5" library="dubec" deviceset="2NMOS" device="30V_0.1A"/>
+<part name="J2" library="dubec" deviceset="M04" device="-929J"/>
+<part name="J3" library="dubec" deviceset="M04" device="-929J"/>
+<part name="J1" library="dubec" deviceset="M04" device="-929J"/>
+<part name="J4" library="dubec" deviceset="M04" device="-929J"/>
 </parts>
 <sheets>
@@
 <wire x1="60.96" y1="81.28" x2="60.96" y2="10.16" width="0.1524" layer="94" style="shortdash"/>
 <text x="12.7" y="86.36" size="3.81" layer="94">Electric Potential Hell</text>
-<wire x1="5.08" y1="-5.08" x2="223.52" y2="-5.08" width="0.1524" layer="94"/>
+<wire x1="5.08" y1="-5.08" x2="215.9" y2="-5.08" width="0.1524" layer="94"/>
 <wire x1="5.08" y1="-91.44" x2="5.08" y2="-5.08" width="0.1524" layer="94"/>
-<wire x1="223.52" y1="-5.08" x2="223.52" y2="-91.44" width="0.1524" layer="94"/>
-<wire x1="223.52" y1="-91.44" x2="5.08" y2="-91.44" width="0.1524" layer="94"/>
+<wire x1="215.9" y1="-5.08" x2="215.9" y2="-91.44" width="0.1524" layer="94"/>
+<wire x1="215.9" y1="-91.44" x2="5.08" y2="-91.44" width="0.1524" layer="94"/>
 <wire x1="142.24" y1="10.16" x2="142.24" y2="91.44" width="0.1524" layer="94" style="shortdash"/>
 <wire x1="233.68" y1="10.16" x2="233.68" y2="91.44" width="0.1524" layer="94" style="shortdash"/>
@@
 <instance part="D2" gate="G$1" x="35.56" y="73.66" rot="R90"/>
 <instance part="D2" gate="G$2" x="27.94" y="53.34" rot="R90"/>
+<instance part="J2" gate="G$1" x="264.16" y="-45.72" rot="R270"/>
+<instance part="J3" gate="G$1" x="261.62" y="-27.94" rot="R90"/>
+<instance part="J1" gate="G$1" x="243.84" y="-45.72" rot="R270"/>
+<instance part="J4" gate="G$1" x="241.3" y="-27.94" rot="R90"/>
 </instances>
 <busses>
@@
 <wire x1="76.2" y1="-78.74" x2="76.2" y2="-81.28" width="0.1524" layer="91"/>
 </segment>
+<segment>
+<label x="238.76" y="-50.8" size="1.27" layer="95" rot="R270" xref="yes"/>
+<pinref part="J1" gate="G$1" pin="1"/>
+<wire x1="238.76" y1="-50.8" x2="238.76" y2="-48.26" width="0.1524" layer="91"/>
+</segment>
+<segment>
+<pinref part="J2" gate="G$1" pin="1"/>
+<wire x1="259.08" y1="-48.26" x2="259.08" y2="-50.8" width="0.1524" layer="91"/>
+<label x="259.08" y="-50.8" size="1.27" layer="95" rot="R270" xref="yes"/>
+</segment>
+<segment>
+<label x="266.7" y="-22.86" size="1.27" layer="95" rot="R90" xref="yes"/>
+<pinref part="J3" gate="G$1" pin="1"/>
+<wire x1="266.7" y1="-22.86" x2="266.7" y2="-25.4" width="0.1524" layer="91"/>
+</segment>
+<segment>
+<pinref part="J4" gate="G$1" pin="1"/>
+<wire x1="246.38" y1="-25.4" x2="246.38" y2="-22.86" width="0.1524" layer="91"/>
+<label x="246.38" y="-22.86" size="1.27" layer="95" rot="R90" xref="yes"/>
+</segment>
 </net>
 <net name="S+" class="0">
@@
 <pinref part="R9" gate="G$1" pin="1"/>
 </segment>
+<segment>
+<pinref part="J4" gate="G$1" pin="2"/>
+<wire x1="243.84" y1="-25.4" x2="243.84" y2="-22.86" width="0.1524" layer="91"/>
+<label x="243.84" y="-22.86" size="1.27" layer="95" rot="R90" xref="yes"/>
+</segment>
 </net>
 <net name="BATT-" class="0">
@@
 <wire x1="43.18" y1="53.34" x2="43.18" y2="50.8" width="0.1524" layer="91"/>
 <label x="43.18" y="50.8" size="1.778" layer="95" rot="R270" xref="yes"/>
+</segment>
+<segment>
+<label x="241.3" y="-50.8" size="1.27" layer="95" rot="R270" xref="yes"/>
+<pinref part="J1" gate="G$1" pin="2"/>
+<wire x1="241.3" y1="-50.8" x2="241.3" y2="-48.26" width="0.1524" layer="91"/>
 </segment>
 </net>
@@
 <wire x1="152.4" y1="-27.94" x2="152.4" y2="-38.1" width="0.1524" layer="91"/>
 <pinref part="U6" gate="G$1" pin="VS"/>
-<wire x1="203.2" y1="-35.56" x2="210.82" y2="-35.56" width="0.1524" layer="91"/>
+<wire x1="203.2" y1="-35.56" x2="208.28" y2="-35.56" width="0.1524" layer="91"/>
 <label x="187.96" y="-66.04" size="1.778" layer="95" rot="R270" xref="yes"/>
 <pinref part="U6" gate="G$1" pin="GND"/>
 <wire x1="187.96" y1="-58.42" x2="187.96" y2="-63.5" width="0.1524" layer="91"/>
-<wire x1="187.96" y1="-63.5" x2="210.82" y2="-63.5" width="0.1524" layer="91"/>
-<wire x1="210.82" y1="-63.5" x2="210.82" y2="-35.56" width="0.1524" layer="91"/>
+<wire x1="187.96" y1="-63.5" x2="208.28" y2="-63.5" width="0.1524" layer="91"/>
+<wire x1="208.28" y1="-63.5" x2="208.28" y2="-35.56" width="0.1524" layer="91"/>
 <wire x1="187.96" y1="-63.5" x2="187.96" y2="-66.04" width="0.1524" layer="91"/>
 <junction x="187.96" y="-63.5"/>
@@
 <segment>
 <pinref part="T1" gate="G$1" pin="2"/>
-<label x="208.28" y="-25.4" size="1.778" layer="95" xref="yes"/>
+<label x="203.2" y="-25.4" size="1.778" layer="95" xref="yes"/>
 <pinref part="U6" gate="G$1" pin="VCC"/>
 <wire x1="187.96" y1="-27.94" x2="187.96" y2="-25.4" width="0.1524" layer="91"/>
-<wire x1="187.96" y1="-25.4" x2="208.28" y2="-25.4" width="0.1524" layer="91"/>
+<wire x1="187.96" y1="-25.4" x2="203.2" y2="-25.4" width="0.1524" layer="91"/>
 <junction x="187.96" y="-25.4"/>
 <pinref part="C10" gate="G$1" pin="2"/>
@@
 <label x="25.4" y="-20.32" size="1.778" layer="95" rot="R180" xref="yes"/>
 <pinref part="C3" gate="G$1" pin="2"/>
+</segment>
+<segment>
+<pinref part="J4" gate="G$1" pin="3"/>
+<wire x1="241.3" y1="-25.4" x2="241.3" y2="-22.86" width="0.1524" layer="91"/>
+<label x="241.3" y="-22.86" size="1.27" layer="95" rot="R90" xref="yes"/>
 </segment>
 </net>
@@
 <wire x1="48.26" y1="-38.1" x2="48.26" y2="-40.64" width="0.1524" layer="91"/>
 <junction x="48.26" y="-38.1"/>
+<label x="88.9" y="-38.1" size="1.778" layer="95" rot="R90" xref="yes"/>
+</segment>
+<segment>
+<pinref part="J4" gate="G$1" pin="4"/>
+<wire x1="238.76" y1="-25.4" x2="238.76" y2="-22.86" width="0.1524" layer="91"/>
+<label x="238.76" y="-22.86" size="1.27" layer="95" rot="R90" xref="yes"/>
 </segment>
 </net>
@@
 <pinref part="U3" gate="G$1" pin="DS"/>
 </segment>
+<segment>
+<label x="259.08" y="-22.86" size="1.27" layer="95" rot="R90" xref="yes"/>
+<pinref part="J3" gate="G$1" pin="4"/>
+<wire x1="259.08" y1="-22.86" x2="259.08" y2="-25.4" width="0.1524" layer="91"/>
+</segment>
 </net>
 <net name="!OE" class="0">
@@
 <label x="248.92" y="40.64" size="1.778" layer="95" rot="R180" xref="yes"/>
 </segment>
+<segment>
+<label x="264.16" y="-22.86" size="1.27" layer="95" rot="R90" xref="yes"/>
+<pinref part="J3" gate="G$1" pin="2"/>
+<wire x1="264.16" y1="-22.86" x2="264.16" y2="-25.4" width="0.1524" layer="91"/>
+</segment>
 </net>
 <net name="CP" class="0">
@@
 <pinref part="U3" gate="G$1" pin="SHCP"/>
 </segment>
-</net>
-<net name="N$19" class="0">
+<segment>
+<label x="261.62" y="-22.86" size="1.27" layer="95" rot="R90" xref="yes"/>
+<pinref part="J3" gate="G$1" pin="3"/>
+<wire x1="261.62" y1="-22.86" x2="261.62" y2="-25.4" width="0.1524" layer="91"/>
+</segment>
+</net>
+<net name="Q7S" class="0">
 <segment>
 <pinref part="U3" gate="G$1" pin="Q7S"/>
 <wire x1="256.54" y1="33.02" x2="254" y2="33.02" width="0.1524" layer="91"/>
 <label x="254" y="33.02" size="1.778" layer="95" rot="R180" xref="yes"/>
+</segment>
+<segment>
+<label x="246.38" y="-50.8" size="1.27" layer="95" rot="R270" xref="yes"/>
+<pinref part="J1" gate="G$1" pin="4"/>
+<wire x1="246.38" y1="-50.8" x2="246.38" y2="-48.26" width="0.1524" layer="91"/>
 </segment>
 </net>
@@
 <label x="129.54" y="-63.5" size="1.778" layer="95" rot="R270" xref="yes"/>
 </segment>
+<segment>
+<label x="266.7" y="-50.8" size="1.27" layer="95" rot="R270" xref="yes"/>
+<pinref part="J2" gate="G$1" pin="4"/>
+<wire x1="266.7" y1="-50.8" x2="266.7" y2="-48.26" width="0.1524" layer="91"/>
+</segment>
 </net>
 <net name="OPTO_A" class="0">
@@
 <wire x1="144.78" y1="-58.42" x2="139.7" y2="-58.42" width="0.1524" layer="91"/>
 <label x="139.7" y="-58.42" size="1.778" layer="95" rot="R90" xref="yes"/>
+</segment>
+<segment>
+<label x="261.62" y="-50.8" size="1.27" layer="95" rot="R270" xref="yes"/>
+<pinref part="J2" gate="G$1" pin="2"/>
+<wire x1="261.62" y1="-50.8" x2="261.62" y2="-48.26" width="0.1524" layer="91"/>
 </segment>
 </net>
@@
 <label x="139.7" y="-63.5" size="1.778" layer="95" rot="R270" xref="yes"/>
 </segment>
-</net>
-<net name="N$30" class="0">
+<segment>
+<label x="264.16" y="-50.8" size="1.27" layer="95" rot="R270" xref="yes"/>
+<pinref part="J2" gate="G$1" pin="3"/>
+<wire x1="264.16" y1="-50.8" x2="264.16" y2="-48.26" width="0.1524" layer="91"/>
+</segment>
+</net>
+<net name="SFB" class="0">
 <segment>
 <pinref part="Q5" gate="G$2" pin="G"/>
@@
 <wire x1="205.74" y1="-50.8" x2="203.2" y2="-50.8" width="0.1524" layer="91"/>
 </segment>
-</net>
+<segment>
+<label x="243.84" y="-50.8" size="1.27" layer="95" rot="R270" xref="yes"/>
+<pinref part="J1" gate="G$1" pin="3"/>
+<wire x1="243.84" y1="-50.8" x2="243.84" y2="-48.26" width="0.1524" layer="91"/>
+</segment>
+</net>
