File: lipovsky-power.sch (EAGLE design)
At the start: 101 parts, among them J1 M04-929J, J2 M04-929J, J3 M04-929J, J4 M04-929J, Q1 NMOS30V_30A, Q11 NMOS40V_10A, Q12 NMOS40V_10A, Q14 NMOS40V_10A, Q15 NMOS40V_10A, Q16 NMOS40V_10A, Q18 NMOS40V_10A, Q2 2NMOS30V_0.1A, Q21 PMOS30V_11A, Q22 PMOS30V_11A, Q23 NMOS40V_10A, Q24 NMOS40V_10A, Q25 PMOS30V_11A, Q26 PMOS30V_11A, Q27 NMOS40V_10A, Q28 NMOS40V_10A, Q3 2PMOS50V_0.17A, Q31 PMOS30V_11A, Q32 PMOS30V_11A, Q33 PMOS30V_11A, Q34 PMOS30V_11A, Q35 PMOS30V_11A, Q36 PMOS30V_11A, Q37 PMOS30V_11A, Q38 PMOS30V_11A, Q4 2PMOS50V_0.17A, Q41 PMOS30V_11A, Q42 PMOS30V_11A, Q43 PMOS30V_11A, Q44 PMOS30V_11A, Q45 PMOS30V_11A, Q46 PMOS30V_11A, Q47 PMOS30V_11A, Q48 PMOS30V_11A, Q5 2NMOS30V_0.1A, Q51 PMOS30V_11A, Q52 PMOS30V_11A, Q53 PMOS30V_11A, Q54 PMOS30V_11A, Q55 PMOS30V_11A, Q56 PMOS30V_11A, Q57 PMOS30V_11A, Q58 PMOS30V_11A, Q62 PMOS30V_11A, Q64 PMOS30V_11A, Q66 PMOS30V_11A, Q68 PMOS30V_11A, T1 TFORM_4_4311_4A4, U1 DG508BEN-T1-GE4, U2 DG508BEN-T1-GE4, U3 74HC595, U4 LTC3805-5IDD, U5 TC1240A, U6 AR30N60PPA-13

Commit message: .
Parts:
- removed C1, C3: CAP4.7U_10V, dubec:CAP4.7U_10V
- removed U5: TC1240A, dubec:TC1240A
Connections:
- removed net N$8: C1.2, U5.C+
- removed net N$9: C1.1, U5.C-
- net S-: no longer U5.GND, U5.SHDN
- net VCC: no longer C3.2, U5.VIN
- net VCC_REG: no longer C3.1, U5.VOUT
Other:
- moved on the sheet: C10, C2, C4, C5, C9, D4, Q1, Q5G$1, Q5G$2, R11, R12, R13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

Commit message: .
Parts:
- removed Q11, Q15: NMOS40V_10A, dubec:NMOS40V_10A
Connections:
- removed net SS+1: Q11.S, Q12.S
- removed net ST+1: Q15.S, Q16.S
- net C1: now also Q12.S, Q16.S; no longer Q11.D, Q15.D
- net GS1: no longer Q11.G
- net GT1: no longer Q15.G
Changed lines of the file:
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@@
 <part name="R2" library="dubec" deviceset="RES" device="4.22K_16"/>
 <part name="T1" library="dubec" deviceset="TFORM_4_4" device="311_4A4"/>
-<part name="Q11" library="dubec" deviceset="NMOS" device="40V_10A"/>
 <part name="Q12" library="dubec" deviceset="NMOS" device="40V_10A"/>
 <part name="Q23" library="dubec" deviceset="NMOS" device="40V_10A"/>
@@
 <part name="Q27" library="dubec" deviceset="NMOS" device="40V_10A"/>
 <part name="Q28" library="dubec" deviceset="NMOS" device="40V_10A"/>
-<part name="Q15" library="dubec" deviceset="NMOS" device="40V_10A"/>
 <part name="Q16" library="dubec" deviceset="NMOS" device="40V_10A"/>
 <part name="RGT6" library="dubec" deviceset="RES" device="100K_16"/>
@@
 <instance part="R2" gate="G$1" x="-20.32" y="-48.26" rot="R90"/>
 <instance part="T1" gate="G$1" x="121.92" y="-27.94" rot="MR0"/>
-<instance part="Q11" gate="G$1" x="-101.6" y="-43.18" rot="R90"/>
 <instance part="Q12" gate="G$1" x="-86.36" y="-43.18" rot="MR90"/>
 <instance part="Q23" gate="G$1" x="-101.6" y="-35.56" rot="MR270"/>
@@
 <instance part="Q27" gate="G$1" x="-45.72" y="-35.56" rot="MR270"/>
 <instance part="Q28" gate="G$1" x="-30.48" y="-35.56" rot="R270"/>
-<instance part="Q15" gate="G$1" x="-45.72" y="-43.18" rot="R90"/>
 <instance part="Q16" gate="G$1" x="-30.48" y="-43.18" rot="MR90"/>
 <instance part="RGT6" gate="G$1" x="167.64" y="71.12"/>
@@
 <wire x1="-111.76" y1="-35.56" x2="-111.76" y2="-43.18" width="0.1524" layer="91"/>
 <wire x1="-111.76" y1="-5.08" x2="-119.38" y2="-5.08" width="0.1524" layer="91"/>
-<pinref part="Q11" gate="G$1" pin="D"/>
-<wire x1="-106.68" y1="-43.18" x2="-111.76" y2="-43.18" width="0.1524" layer="91"/>
 <pinref part="Q23" gate="G$1" pin="D"/>
 <wire x1="-111.76" y1="-35.56" x2="-106.68" y2="-35.56" width="0.1524" layer="91"/>
 <junction x="-111.76" y="-35.56"/>
+<pinref part="Q12" gate="G$1" pin="S"/>
+<wire x1="-111.76" y1="-43.18" x2="-91.44" y2="-43.18" width="0.1524" layer="91"/>
 </segment>
 <segment>
@@
 <wire x1="-55.88" y1="-35.56" x2="-55.88" y2="-43.18" width="0.1524" layer="91"/>
 <junction x="-55.88" y="-35.56"/>
-<wire x1="-55.88" y1="-43.18" x2="-50.8" y2="-43.18" width="0.1524" layer="91"/>
 <label x="-63.5" y="-5.08" size="1.27" layer="95" rot="R180" xref="yes"/>
 <pinref part="Q27" gate="G$1" pin="D"/>
-<pinref part="Q15" gate="G$1" pin="D"/>
+<pinref part="Q16" gate="G$1" pin="S"/>
+<wire x1="-55.88" y1="-43.18" x2="-35.56" y2="-43.18" width="0.1524" layer="91"/>
 </segment>
 </net>
@@
 <pinref part="Q14" gate="G$1" pin="G"/>
 <pinref part="Q12" gate="G$1" pin="G"/>
-<label x="-93.98" y="-48.26" size="1.27" layer="95" rot="R90" xref="yes"/>
-<pinref part="Q11" gate="G$1" pin="G"/>
-<wire x1="-99.06" y1="-48.26" x2="-88.9" y2="-48.26" width="0.1524" layer="91"/>
+<label x="-93.98" y="-48.26" size="1.27" layer="95" rot="R180" xref="yes"/>
+<wire x1="-93.98" y1="-48.26" x2="-88.9" y2="-48.26" width="0.1524" layer="91"/>
 <junction x="-88.9" y="-48.26"/>
 </segment>
@@
 </segment>
 </net>
-<net name="SS+1" class="0">
-<segment>
-<pinref part="Q12" gate="G$1" pin="S"/>
-<pinref part="Q11" gate="G$1" pin="S"/>
-<wire x1="-96.52" y1="-43.18" x2="-91.44" y2="-43.18" width="0.1524" layer="91"/>
-</segment>
-</net>
 <net name="C4+" class="0">
 <segment>
@@
 <pinref part="Q16" gate="G$1" pin="G"/>
 <pinref part="Q18" gate="G$1" pin="G"/>
-<pinref part="Q15" gate="G$1" pin="G"/>
-<wire x1="-33.02" y1="-48.26" x2="-43.18" y2="-48.26" width="0.1524" layer="91"/>
+<wire x1="-33.02" y1="-48.26" x2="-38.1" y2="-48.26" width="0.1524" layer="91"/>
 <junction x="-33.02" y="-48.26"/>
-<label x="-38.1" y="-48.26" size="1.27" layer="95" rot="R90" xref="yes"/>
+<label x="-38.1" y="-48.26" size="1.27" layer="95" rot="R180" xref="yes"/>
 </segment>
 <segment>
@@
 </segment>
 </net>
-<net name="ST+1" class="0">
-<segment>
-<pinref part="Q15" gate="G$1" pin="S"/>
-<pinref part="Q16" gate="G$1" pin="S"/>
-<wire x1="-40.64" y1="-43.18" x2="-35.56" y2="-43.18" width="0.1524" layer="91"/>
-</segment>
-</net>

Commit message: .
Parts:
- added R9: RES5.9K_16, dubec:RES5.9K_16
- R17: value RES402_16 -> RES330_16; device dubec:RES402_16 -> dubec:RES330_16
- R18: value RES5.1K_16 -> RES1K_16; device dubec:RES5.1K_16 -> dubec:RES1K_16
Connections:
- net RUN_REG renamed EN_FLYBACK
- net VCC renamed +5V
- net VCC_REG renamed +8V
- new net N$4: R9.1, U4.OC
- net S-: no longer U4.OC
- net SENSE: now also R9.2
- net SFB: no longer J1.3
Changed lines of the file:
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@@
 <part name="R15" library="dubec" deviceset="RES" device="100K_16"/>
 <part name="C10" library="dubec" deviceset="CAP" device="47UF_10V"/>
-<part name="R17" library="dubec" deviceset="RES" device="402_16"/>
-<part name="R18" library="dubec" deviceset="RES" device="5.1K_16"/>
+<part name="R17" library="dubec" deviceset="RES" device="330_16" value="RES330_16"/>
+<part name="R18" library="dubec" deviceset="RES" device="1K_16" value="RES1K_16"/>
 <part name="Q5" library="dubec" deviceset="2NMOS" device="30V_0.1A"/>
 <part name="J2" library="dubec" deviceset="M04" device="-929J"/>
@@
 <part name="J1" library="dubec" deviceset="M04" device="-929J"/>
 <part name="J4" library="dubec" deviceset="M04" device="-929J"/>
+<part name="R9" library="dubec" deviceset="RES" device="5.9K_16"/>
 </parts>
 <sheets>
@@
 <instance part="J1" gate="G$1" x="243.84" y="-45.72" rot="R270"/>
 <instance part="J4" gate="G$1" x="241.3" y="-27.94" rot="R90"/>
+<instance part="R9" gate="G$1" x="86.36" y="-55.88"/>
 </instances>
 <busses>
@@
 <wire x1="86.36" y1="-71.12" x2="86.36" y2="-78.74" width="0.1524" layer="91"/>
 <junction x="86.36" y="-78.74"/>
-<wire x1="81.28" y1="-78.74" x2="86.36" y2="-78.74" width="0.1524" layer="91"/>
-<pinref part="U4" gate="G$1" pin="OC"/>
-<wire x1="78.74" y1="-53.34" x2="81.28" y2="-53.34" width="0.1524" layer="91"/>
-<wire x1="81.28" y1="-53.34" x2="81.28" y2="-78.74" width="0.1524" layer="91"/>
-<wire x1="63.5" y1="-78.74" x2="81.28" y2="-78.74" width="0.1524" layer="91"/>
+<wire x1="63.5" y1="-78.74" x2="86.36" y2="-78.74" width="0.1524" layer="91"/>
 <junction x="63.5" y="-78.74"/>
-<junction x="81.28" y="-78.74"/>
 <pinref part="U4" gate="G$1" pin="GND"/>
 <wire x1="63.5" y1="-78.74" x2="63.5" y2="-71.12" width="0.1524" layer="91"/>
@@
 </segment>
 </net>
-<net name="VCC" class="0">
+<net name="+5V" class="0">
 <segment>
 <pinref part="U3" gate="G$1" pin="VCC"/>
@@
 </segment>
 </net>
-<net name="VCC_REG" class="0">
+<net name="+8V" class="0">
 <segment>
 <wire x1="27.94" y1="-38.1" x2="33.02" y2="-38.1" width="0.1524" layer="91"/>
@@
 <pinref part="Q1" gate="G$1" pin="S"/>
 <pinref part="R5" gate="G$1" pin="2"/>
-<wire x1="91.44" y1="-50.8" x2="91.44" y2="-58.42" width="0.1524" layer="91"/>
+<wire x1="91.44" y1="-50.8" x2="91.44" y2="-55.88" width="0.1524" layer="91"/>
 <pinref part="R8" gate="G$1" pin="2"/>
+<wire x1="91.44" y1="-55.88" x2="91.44" y2="-58.42" width="0.1524" layer="91"/>
 <wire x1="91.44" y1="-58.42" x2="91.44" y2="-66.04" width="0.1524" layer="91"/>
 <wire x1="88.9" y1="-58.42" x2="91.44" y2="-58.42" width="0.1524" layer="91"/>
 <junction x="91.44" y="-58.42"/>
+<pinref part="R9" gate="G$1" pin="2"/>
+<wire x1="88.9" y1="-55.88" x2="91.44" y2="-55.88" width="0.1524" layer="91"/>
+<junction x="91.44" y="-55.88"/>
 </segment>
 </net>
@@
 </segment>
 </net>
-<net name="RUN_REG" class="0">
+<net name="EN_FLYBACK" class="0">
 <segment>
 <pinref part="U4" gate="G$1" pin="RUN"/>
@@
 <wire x1="193.04" y1="-50.8" x2="190.5" y2="-50.8" width="0.1524" layer="91"/>
 </segment>
-<segment>
-<label x="243.84" y="-50.8" size="1.27" layer="95" rot="R270" xref="yes"/>
-<pinref part="J1" gate="G$1" pin="3"/>
-<wire x1="243.84" y1="-50.8" x2="243.84" y2="-48.26" width="0.1524" layer="91"/>
-</segment>
-</net>
+</net>
+<net name="N$4" class="0">
+<segment>
+<pinref part="U4" gate="G$1" pin="OC"/>
+<wire x1="78.74" y1="-53.34" x2="81.28" y2="-53.34" width="0.1524" layer="91"/>
+<wire x1="81.28" y1="-53.34" x2="81.28" y2="-55.88" width="0.1524" layer="91"/>
+<pinref part="R9" gate="G$1" pin="1"/>
+<wire x1="81.28" y1="-55.88" x2="83.82" y2="-55.88" width="0.1524" layer="91"/>
+</segment>
+</net>

Commit message: .
Connections:
- net BATT-: now also D2G$1.A, D2G$1.C, J1.4
- net Q7S: now also J1.3; no longer J1.4
Other:
- moved on the sheet: C10, C2, C4, C5, C9, D2G$1, D4, J1, J2, J3, J4, Q1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

Commit message: .
Connections:
- net BATT-: now also Q2G$1.D, Q2G$1.G, Q2G$1.S, Q3G$2.G, Q3G$2.S; no longer J1.4
- net Q7S: no longer J1.3
- net T+: now also J1.4
- net T-: now also J1.3
Other:
- moved on the sheet: D2G$1, Q2G$1, Q3G$2

Commit message: .
Connections:
- new net N$8: T1.4
Changed lines of the file:
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@@
+</segment>
+</net>
+<net name="N$8" class="0">
+<segment>
+<pinref part="T1" gate="G$1" pin="4"/>
+<wire x1="119.38" y1="-33.02" x2="121.92" y2="-33.02" width="0.1524" layer="91"/>
 </segment>
 </net>

Commit message: .
Parts:
- added U$2: JUMPER-PAD, dubec:JUMPER-PAD
- R3: value RES4.7K_16 -> RES10K_16; device dubec:RES4.7K_16 -> dubec:RES10K_16
Connections:
- new net N$7: T1.3, U$2.2
- net T-: now also U$2.1; no longer T1.3
Changed lines of the file:
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@@
 <part name="RGT-2" library="dubec" deviceset="RES" device="100K_16"/>
 <part name="U3" library="dubec" deviceset="74HC595" device=""/>
-<part name="R3" library="dubec" deviceset="RES" device="4.7K_16" value="RES4.7K_16"/>
+<part name="R3" library="dubec" deviceset="RES" device="10K_16" value="RES10K_16"/>
 <part name="R4" library="dubec" deviceset="RES" device="4.7K_16" value="RES4.7K_16"/>
 <part name="Q1" library="dubec" deviceset="NMOS" device="30V_30A"/>
@@
 <part name="J4" library="dubec" deviceset="M04" device="-929J"/>
 <part name="R9" library="dubec" deviceset="RES" device="5.9K_16"/>
+<part name="U$2" library="dubec" deviceset="JUMPER-PAD" device=""/>
 </parts>
 <sheets>
@@
 <wire x1="60.96" y1="81.28" x2="60.96" y2="10.16" width="0.1524" layer="94" style="shortdash"/>
 <text x="12.7" y="86.36" size="3.81" layer="94">Electric Potential Hell</text>
-<wire x1="5.08" y1="-5.08" x2="190.5" y2="-5.08" width="0.1524" layer="94"/>
+<wire x1="5.08" y1="-5.08" x2="195.58" y2="-5.08" width="0.1524" layer="94"/>
 <wire x1="5.08" y1="-91.44" x2="5.08" y2="-5.08" width="0.1524" layer="94"/>
-<wire x1="190.5" y1="-5.08" x2="190.5" y2="-91.44" width="0.1524" layer="94"/>
-<wire x1="190.5" y1="-91.44" x2="5.08" y2="-91.44" width="0.1524" layer="94"/>
+<wire x1="195.58" y1="-5.08" x2="195.58" y2="-91.44" width="0.1524" layer="94"/>
+<wire x1="195.58" y1="-91.44" x2="5.08" y2="-91.44" width="0.1524" layer="94"/>
 <wire x1="142.24" y1="10.16" x2="142.24" y2="91.44" width="0.1524" layer="94" style="shortdash"/>
 <wire x1="233.68" y1="10.16" x2="233.68" y2="91.44" width="0.1524" layer="94" style="shortdash"/>
@@
 <instance part="J4" gate="G$1" x="220.98" y="-22.86" rot="R90"/>
 <instance part="R9" gate="G$1" x="78.74" y="-55.88"/>
+<instance part="U$2" gate="G$1" x="127" y="-33.02" rot="R90"/>
 </instances>
 <busses>
@@
 </segment>
 <segment>
-<pinref part="T1" gate="G$1" pin="3"/>
-<wire x1="127" y1="-27.94" x2="119.38" y2="-27.94" width="0.1524" layer="91"/>
-<wire x1="127" y1="-27.94" x2="127" y2="-38.1" width="0.1524" layer="91"/>
 <pinref part="U6" gate="G$1" pin="VS"/>
 <wire x1="172.72" y1="-35.56" x2="177.8" y2="-35.56" width="0.1524" layer="91"/>
-<label x="157.48" y="-66.04" size="1.778" layer="95" rot="R270" xref="yes"/>
+<label x="182.88" y="-63.5" size="1.778" layer="95" xref="yes"/>
 <pinref part="U6" gate="G$1" pin="GND"/>
 <wire x1="157.48" y1="-58.42" x2="157.48" y2="-63.5" width="0.1524" layer="91"/>
 <wire x1="157.48" y1="-63.5" x2="177.8" y2="-63.5" width="0.1524" layer="91"/>
 <wire x1="177.8" y1="-63.5" x2="177.8" y2="-35.56" width="0.1524" layer="91"/>
-<wire x1="157.48" y1="-63.5" x2="157.48" y2="-66.04" width="0.1524" layer="91"/>
 <junction x="157.48" y="-63.5"/>
 <pinref part="R14" gate="G$1" pin="1"/>
@@
 <wire x1="137.16" y1="-68.58" x2="139.7" y2="-68.58" width="0.1524" layer="91"/>
 <wire x1="139.7" y1="-68.58" x2="139.7" y2="-63.5" width="0.1524" layer="91"/>
+<pinref part="U$2" gate="G$1" pin="1"/>
+<wire x1="177.8" y1="-63.5" x2="182.88" y2="-63.5" width="0.1524" layer="91"/>
+<junction x="177.8" y="-63.5"/>
 </segment>
 <segment>
@@
 <segment>
 <pinref part="T1" gate="G$1" pin="2"/>
-<label x="177.8" y="-25.4" size="1.778" layer="95" xref="yes"/>
+<label x="182.88" y="-25.4" size="1.778" layer="95" xref="yes"/>
 <pinref part="U6" gate="G$1" pin="VCC"/>
 <wire x1="157.48" y1="-27.94" x2="157.48" y2="-25.4" width="0.1524" layer="91"/>
-<wire x1="157.48" y1="-25.4" x2="177.8" y2="-25.4" width="0.1524" layer="91"/>
+<wire x1="157.48" y1="-25.4" x2="182.88" y2="-25.4" width="0.1524" layer="91"/>
 <junction x="157.48" y="-25.4"/>
 <pinref part="C10" gate="G$1" pin="2"/>
@@
 </segment>
 </net>
+<net name="N$7" class="0">
+<segment>
+<pinref part="U$2" gate="G$1" pin="2"/>
+<pinref part="T1" gate="G$1" pin="3"/>
+<wire x1="127" y1="-27.94" x2="119.38" y2="-27.94" width="0.1524" layer="91"/>
+</segment>
+</net>

Commit message: tweaks
Parts:
- R3: value RES10K_16 -> RES12K_16; device dubec:RES10K_16 -> dubec:RES12K_16
- RGS+2, RGS-2, RGS1, RGS3, RGS4, RGS5, RGS6, RGT+2, RGT-2, RGT1, RGT3, RGT4, RGT5, RGT6: value RES100K_16 -> RES12K_16; device dubec:RES100K_16 -> dubec:RES12K_16
Changed lines of the file:
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@@
 <parts>
 <part name="JP1" library="dubec" deviceset="M07" device="XHRA" value="M07XHRA"/>
-<part name="RGS6" library="dubec" deviceset="RES" device="100K_16"/>
-<part name="RGS5" library="dubec" deviceset="RES" device="100K_16"/>
-<part name="RGS4" library="dubec" deviceset="RES" device="100K_16"/>
-<part name="RGS3" library="dubec" deviceset="RES" device="100K_16"/>
-<part name="RGS+2" library="dubec" deviceset="RES" device="100K_16"/>
+<part name="RGS6" library="dubec" deviceset="RES" device="12K_16" value="RES12K_16"/>
+<part name="RGS5" library="dubec" deviceset="RES" device="12K_16" value="RES12K_16"/>
+<part name="RGS4" library="dubec" deviceset="RES" device="12K_16" value="RES12K_16"/>
+<part name="RGS3" library="dubec" deviceset="RES" device="12K_16" value="RES12K_16"/>
+<part name="RGS+2" library="dubec" deviceset="RES" device="12K_16" value="RES12K_16"/>
 <part name="Q21" library="dubec" deviceset="PMOS" device="30V_11A"/>
 <part name="Q22" library="dubec" deviceset="PMOS" device="30V_11A"/>
@@
 <part name="Q23" library="dubec" deviceset="NMOS" device="40V_10A"/>
 <part name="Q24" library="dubec" deviceset="NMOS" device="40V_10A"/>
-<part name="RGS1" library="dubec" deviceset="RES" device="100K_16"/>
-<part name="RGS-2" library="dubec" deviceset="RES" device="100K_16"/>
+<part name="RGS1" library="dubec" deviceset="RES" device="12K_16" value="RES12K_16"/>
+<part name="RGS-2" library="dubec" deviceset="RES" device="12K_16" value="RES12K_16"/>
 <part name="Q2" library="dubec" deviceset="2NMOS" device="30V_0.1A"/>
 <part name="Q27" library="dubec" deviceset="NMOS" device="40V_10A"/>
 <part name="Q28" library="dubec" deviceset="NMOS" device="40V_10A"/>
 <part name="Q16" library="dubec" deviceset="NMOS" device="40V_10A"/>
-<part name="RGT6" library="dubec" deviceset="RES" device="100K_16"/>
-<part name="RGT5" library="dubec" deviceset="RES" device="100K_16"/>
-<part name="RGT4" library="dubec" deviceset="RES" device="100K_16"/>
-<part name="RGT3" library="dubec" deviceset="RES" device="100K_16"/>
-<part name="RGT+2" library="dubec" deviceset="RES" device="100K_16"/>
-<part name="RGT1" library="dubec" deviceset="RES" device="100K_16"/>
-<part name="RGT-2" library="dubec" deviceset="RES" device="100K_16"/>
+<part name="RGT6" library="dubec" deviceset="RES" device="12K_16" value="RES12K_16"/>
+<part name="RGT5" library="dubec" deviceset="RES" device="12K_16" value="RES12K_16"/>
+<part name="RGT4" library="dubec" deviceset="RES" device="12K_16" value="RES12K_16"/>
+<part name="RGT3" library="dubec" deviceset="RES" device="12K_16" value="RES12K_16"/>
+<part name="RGT+2" library="dubec" deviceset="RES" device="12K_16" value="RES12K_16"/>
+<part name="RGT1" library="dubec" deviceset="RES" device="12K_16" value="RES12K_16"/>
+<part name="RGT-2" library="dubec" deviceset="RES" device="12K_16" value="RES12K_16"/>
 <part name="U3" library="dubec" deviceset="74HC595" device=""/>
-<part name="R3" library="dubec" deviceset="RES" device="10K_16" value="RES10K_16"/>
+<part name="R3" library="dubec" deviceset="RES" device="12K_16" value="RES12K_16"/>
 <part name="R4" library="dubec" deviceset="RES" device="4.7K_16" value="RES4.7K_16"/>
 <part name="Q1" library="dubec" deviceset="NMOS" device="30V_30A"/>
@@
 <wire x1="121.92" y1="81.28" x2="124.46" y2="81.28" width="0.1524" layer="91"/>
 <label x="124.46" y="81.28" size="1.778" layer="95" xref="yes"/>
-</segment>
-<segment>
+<wire x1="121.92" y1="81.28" x2="121.92" y2="78.74" width="0.1524" layer="91"/>
+<junction x="121.92" y="81.28"/>
+<wire x1="121.92" y1="78.74" x2="116.84" y2="78.74" width="0.1524" layer="91"/>
+<wire x1="116.84" y1="78.74" x2="116.84" y2="73.66" width="0.1524" layer="91"/>
+<wire x1="116.84" y1="73.66" x2="121.92" y2="73.66" width="0.1524" layer="91"/>
 <pinref part="U1" gate="G$1" pin="D"/>
-<wire x1="121.92" y1="71.12" x2="124.46" y2="71.12" width="0.1524" layer="91"/>
-<label x="124.46" y="71.12" size="1.778" layer="95" xref="yes"/>
-<wire x1="121.92" y1="71.12" x2="121.92" y2="68.58" width="0.1524" layer="91"/>
-<junction x="121.92" y="71.12"/>
-<wire x1="121.92" y1="68.58" x2="101.6" y2="68.58" width="0.1524" layer="91"/>
 <pinref part="U1" gate="G$1" pin="S8"/>
 <pinref part="U1" gate="G$1" pin="S7"/>
@@
 <pinref part="U1" gate="G$1" pin="S6"/>
 <junction x="101.6" y="76.2"/>
-<wire x1="101.6" y1="76.2" x2="101.6" y2="71.12" width="0.1524" layer="91"/>
-<wire x1="101.6" y1="68.58" x2="101.6" y2="71.12" width="0.1524" layer="91"/>
-<junction x="101.6" y="71.12"/>
-</segment>
-<segment>
+<wire x1="101.6" y1="76.2" x2="101.6" y2="73.66" width="0.1524" layer="91"/>
+<wire x1="101.6" y1="73.66" x2="101.6" y2="71.12" width="0.1524" layer="91"/>
+<wire x1="121.92" y1="73.66" x2="121.92" y2="71.12" width="0.1524" layer="91"/>
+<wire x1="116.84" y1="73.66" x2="101.6" y2="73.66" width="0.1524" layer="91"/>
+<junction x="116.84" y="73.66"/>
+<junction x="101.6" y="73.66"/>
+</segment>
+<segment>
