File: lipovsky-control.sch (EAGLE design)
At the start: 41 parts, among them J1 M04-929P, J2 M04-929P, J3 M04-929P, J4 M04-929P, U1 ATTINYX4A8MU, U2 MIC2288YD5, U3 MIC2288YD5, U7 LTV-816S

Commit message: .
Parts:
- added J5: AVRISPWR, dubec:AVRISPWR
- added R15: RES10K_16, dubec:RES10K_16
Connections:
- removed net N$8: R10.2, U1.PA5
- new net N$3: R10.1, U1.PB0
- net !OE: now also J5.SCK, U1.PA4; no longer U1.PB0
- net !RESET: now also J5.RESET, R15.2
- net +5V: now also J5.VCC, R15.1
- net CP: now also J5.MISO, U1.PA5; no longer U1.PB1
- net D1: now also R7.2; no longer R7.1
- net D2: now also R8.2; no longer R8.1
- net D3: now also R9.2; no longer R9.1
- net D4: now also R10.2; no longer R10.1
- net DS: now also J5.MOSI, U1.PA6; no longer U1.PB2
- net D_OVERTEMP: now also U1.PA3; no longer U1.PA7
- net D_STATUS: now also U1.PA2; no longer U1.PA6
- net N$5: now also R8.1, U1.PB2; no longer R7.2, U1.PA2
- net N$6: now also R7.1, U1.PA7; no longer R8.2, U1.PA3
- net N$7: now also R9.1, U1.PB1; no longer R9.2, U1.PA4
- net S-: now also J5.GND
Other:
- moved on the sheet: R10, R7, R8, R9
Changed lines of the file:
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@@
 <part name="R14" library="dubec" deviceset="RES" device="330_16" value="RES330_16"/>
 <part name="C3" library="dubec" deviceset="CAP" device="47N_50V" value="CAP47N_50V"/>
+<part name="J5" library="dubec" deviceset="AVRISP" device="WR"/>
+<part name="R15" library="dubec" deviceset="RES" device="10K_16"/>
 </parts>
 <sheets>
@@
 <instance part="D4" gate="G$1" x="-2.54" y="-22.86"/>
 <instance part="D5" gate="G$1" x="-2.54" y="-38.1"/>
-<instance part="R7" gate="G$1" x="-2.54" y="22.86"/>
-<instance part="R8" gate="G$1" x="-2.54" y="20.32"/>
-<instance part="R9" gate="G$1" x="-2.54" y="17.78"/>
-<instance part="R10" gate="G$1" x="-2.54" y="15.24"/>
+<instance part="R7" gate="G$1" x="27.94" y="25.4"/>
+<instance part="R8" gate="G$1" x="27.94" y="17.78"/>
+<instance part="R9" gate="G$1" x="27.94" y="20.32"/>
+<instance part="R10" gate="G$1" x="27.94" y="22.86"/>
 <instance part="R11" gate="G$1" x="5.08" y="-40.64" rot="R90"/>
 <instance part="R12" gate="G$1" x="10.16" y="-35.56" rot="R180"/>
@@
 <instance part="R14" gate="G$1" x="48.26" y="-27.94"/>
 <instance part="C3" gate="G$1" x="43.18" y="-35.56" rot="R90"/>
+<instance part="J5" gate="G$1" x="111.76" y="22.86"/>
+<instance part="R15" gate="G$1" x="25.4" y="10.16" rot="R90"/>
 </instances>
 <busses>
@@
 <segment>
 <pinref part="U1" gate="G$1" pin="GND"/>
-<wire x1="12.7" y1="10.16" x2="12.7" y2="7.62" width="0.1524" layer="91"/>
-<label x="12.7" y="7.62" size="1.27" layer="95" rot="R270" xref="yes"/>
+<wire x1="12.7" y1="10.16" x2="12.7" y2="5.08" width="0.1524" layer="91"/>
+<label x="12.7" y="5.08" size="1.27" layer="95" rot="R270" xref="yes"/>
 </segment>
 <segment>
@@
 <junction x="0" y="40.64"/>
 </segment>
+<segment>
+<pinref part="J5" gate="G$1" pin="GND"/>
+<wire x1="104.14" y1="27.94" x2="101.6" y2="25.4" width="0.1524" layer="91"/>
+<label x="101.6" y="25.4" size="1.27" layer="95" rot="R180" xref="yes"/>
+</segment>
 </net>
 <net name="OPTO_A" class="0">
@@
 </segment>
 </net>
-<net name="N$5" class="0">
-<segment>
-<pinref part="U1" gate="G$1" pin="PA2"/>
-<wire x1="2.54" y1="22.86" x2="0" y2="22.86" width="0.1524" layer="91"/>
-<pinref part="R7" gate="G$1" pin="2"/>
-</segment>
-</net>
-<net name="N$6" class="0">
-<segment>
-<pinref part="U1" gate="G$1" pin="PA3"/>
-<wire x1="2.54" y1="20.32" x2="0" y2="20.32" width="0.1524" layer="91"/>
-<pinref part="R8" gate="G$1" pin="2"/>
-</segment>
-</net>
-<net name="N$7" class="0">
-<segment>
-<pinref part="U1" gate="G$1" pin="PA4"/>
-<wire x1="2.54" y1="17.78" x2="0" y2="17.78" width="0.1524" layer="91"/>
-<pinref part="R9" gate="G$1" pin="2"/>
-</segment>
-</net>
-<net name="N$8" class="0">
-<segment>
-<pinref part="U1" gate="G$1" pin="PA5"/>
-<wire x1="2.54" y1="15.24" x2="0" y2="15.24" width="0.1524" layer="91"/>
-<pinref part="R10" gate="G$1" pin="2"/>
-</segment>
-</net>
 <net name="!RESET" class="0">
 <segment>
 <pinref part="U1" gate="G$1" pin="PB3"/>
 <wire x1="22.86" y1="15.24" x2="25.4" y2="15.24" width="0.1524" layer="91"/>
-<label x="25.4" y="15.24" size="1.27" layer="95" xref="yes"/>
+<label x="33.02" y="15.24" size="1.27" layer="95" xref="yes"/>
+<pinref part="R15" gate="G$1" pin="2"/>
+<wire x1="25.4" y1="15.24" x2="33.02" y2="15.24" width="0.1524" layer="91"/>
+<wire x1="25.4" y1="15.24" x2="25.4" y2="12.7" width="0.1524" layer="91"/>
+<junction x="25.4" y="15.24"/>
+</segment>
+<segment>
+<pinref part="J5" gate="G$1" pin="RESET"/>
+<wire x1="119.38" y1="27.94" x2="121.92" y2="25.4" width="0.1524" layer="91"/>
+<label x="121.92" y="25.4" size="1.27" layer="95" xref="yes"/>
 </segment>
 </net>
@@
 <label x="55.88" y="-17.78" size="1.778" layer="95" rot="R90" xref="yes"/>
 </segment>
+<segment>
+<pinref part="R15" gate="G$1" pin="1"/>
+<wire x1="25.4" y1="7.62" x2="25.4" y2="5.08" width="0.1524" layer="91"/>
+<label x="25.4" y="5.08" size="1.27" layer="95" rot="R270" xref="yes"/>
+</segment>
+<segment>
+<pinref part="J5" gate="G$1" pin="VCC"/>
+<wire x1="104.14" y1="17.78" x2="101.6" y2="15.24" width="0.1524" layer="91"/>
+<label x="101.6" y="15.24" size="1.27" layer="95" rot="R180" xref="yes"/>
+</segment>
 </net>
 <net name="BATT-" class="0">
@@
 </segment>
 <segment>
-<pinref part="U1" gate="G$1" pin="PB0"/>
-<wire x1="22.86" y1="22.86" x2="25.4" y2="22.86" width="0.1524" layer="91"/>
-<label x="25.4" y="22.86" size="1.27" layer="95" xref="yes"/>
+<label x="-10.16" y="17.78" size="1.27" layer="95" rot="R180" xref="yes"/>
+<pinref part="U1" gate="G$1" pin="PA4"/>
+<wire x1="-10.16" y1="17.78" x2="2.54" y2="17.78" width="0.1524" layer="91"/>
+</segment>
+<segment>
+<pinref part="J5" gate="G$1" pin="SCK"/>
+<wire x1="119.38" y1="22.86" x2="121.92" y2="20.32" width="0.1524" layer="91"/>
+<label x="121.92" y="20.32" size="1.27" layer="95" xref="yes"/>
 </segment>
 </net>
@@
 </segment>
 <segment>
-<pinref part="U1" gate="G$1" pin="PB1"/>
-<wire x1="22.86" y1="20.32" x2="25.4" y2="20.32" width="0.1524" layer="91"/>
-<label x="25.4" y="20.32" size="1.27" layer="95" xref="yes"/>
+<label x="-10.16" y="15.24" size="1.27" layer="95" rot="R180" xref="yes"/>
+<pinref part="U1" gate="G$1" pin="PA5"/>
+<wire x1="-10.16" y1="15.24" x2="2.54" y2="15.24" width="0.1524" layer="91"/>
+</segment>
+<segment>
+<pinref part="J5" gate="G$1" pin="MISO"/>
+<wire x1="119.38" y1="17.78" x2="121.92" y2="15.24" width="0.1524" layer="91"/>
+<label x="121.92" y="15.24" size="1.27" layer="95" xref="yes"/>
 </segment>
 </net>
@@
 </segment>
 <segment>
-<pinref part="U1" gate="G$1" pin="PB2"/>
-<wire x1="22.86" y1="17.78" x2="25.4" y2="17.78" width="0.1524" layer="91"/>
-<label x="25.4" y="17.78" size="1.27" layer="95" xref="yes"/>
+<label x="33.02" y="27.94" size="1.27" layer="95" xref="yes"/>
+<pinref part="U1" gate="G$1" pin="PA6"/>
+<wire x1="33.02" y1="27.94" x2="22.86" y2="27.94" width="0.1524" layer="91"/>
+</segment>
+<segment>
+<pinref part="J5" gate="G$1" pin="MOSI"/>
+<wire x1="104.14" y1="22.86" x2="101.6" y2="20.32" width="0.1524" layer="91"/>
+<label x="101.6" y="20.32" size="1.27" layer="95" rot="R180" xref="yes"/>
 </segment>
 </net>
@@
 </segment>
 <segment>
-<pinref part="R7" gate="G$1" pin="1"/>
-<wire x1="-5.08" y1="22.86" x2="-10.16" y2="22.86" width="0.1524" layer="91"/>
-<label x="-10.16" y="22.86" size="1.27" layer="95" rot="R180" xref="yes"/>
+<label x="33.02" y="25.4" size="1.27" layer="95" xref="yes"/>
+<pinref part="R7" gate="G$1" pin="2"/>
+<wire x1="30.48" y1="25.4" x2="33.02" y2="25.4" width="0.1524" layer="91"/>
 </segment>
 </net>
@@
 </segment>
 <segment>
-<pinref part="R8" gate="G$1" pin="1"/>
-<wire x1="-5.08" y1="20.32" x2="-10.16" y2="20.32" width="0.1524" layer="91"/>
-<label x="-10.16" y="20.32" size="1.27" layer="95" rot="R180" xref="yes"/>
+<label x="33.02" y="17.78" size="1.27" layer="95" xref="yes"/>
+<pinref part="R8" gate="G$1" pin="2"/>
+<wire x1="30.48" y1="17.78" x2="33.02" y2="17.78" width="0.1524" layer="91"/>
 </segment>
 </net>
@@
 </segment>
 <segment>
-<pinref part="R9" gate="G$1" pin="1"/>
-<wire x1="-5.08" y1="17.78" x2="-10.16" y2="17.78" width="0.1524" layer="91"/>
-<label x="-10.16" y="17.78" size="1.27" layer="95" rot="R180" xref="yes"/>
+<label x="33.02" y="20.32" size="1.27" layer="95" xref="yes"/>
+<pinref part="R9" gate="G$1" pin="2"/>
+<wire x1="33.02" y1="20.32" x2="30.48" y2="20.32" width="0.1524" layer="91"/>
 </segment>
 </net>
@@
 </segment>
 <segment>
-<pinref part="R10" gate="G$1" pin="1"/>
-<wire x1="-5.08" y1="15.24" x2="-10.16" y2="15.24" width="0.1524" layer="91"/>
-<label x="-10.16" y="15.24" size="1.27" layer="95" rot="R180" xref="yes"/>
+<label x="33.02" y="22.86" size="1.27" layer="95" xref="yes"/>
+<pinref part="R10" gate="G$1" pin="2"/>
+<wire x1="33.02" y1="22.86" x2="30.48" y2="22.86" width="0.1524" layer="91"/>
 </segment>
 </net>
@@
 </segment>
 <segment>
-<pinref part="U1" gate="G$1" pin="PA6"/>
-<wire x1="22.86" y1="27.94" x2="25.4" y2="27.94" width="0.1524" layer="91"/>
-<label x="25.4" y="27.94" size="1.27" layer="95" xref="yes"/>
+<label x="-10.16" y="22.86" size="1.27" layer="95" rot="R180" xref="yes"/>
+<pinref part="U1" gate="G$1" pin="PA2"/>
+<wire x1="-10.16" y1="22.86" x2="2.54" y2="22.86" width="0.1524" layer="91"/>
 </segment>
 </net>
@@
 </segment>
 <segment>
-<pinref part="U1" gate="G$1" pin="PA7"/>
-<wire x1="22.86" y1="25.4" x2="25.4" y2="25.4" width="0.1524" layer="91"/>
-<label x="25.4" y="25.4" size="1.27" layer="95" xref="yes"/>
+<label x="-10.16" y="20.32" size="1.27" layer="95" rot="R180" xref="yes"/>
+<wire x1="2.54" y1="20.32" x2="-10.16" y2="20.32" width="0.1524" layer="91"/>
+<pinref part="U1" gate="G$1" pin="PA3"/>
 </segment>
 </net>
@@
 </segment>
 </net>
+<net name="N$3" class="0">
+<segment>
+<pinref part="U1" gate="G$1" pin="PB0"/>
+<pinref part="R10" gate="G$1" pin="1"/>
+<wire x1="22.86" y1="22.86" x2="25.4" y2="22.86" width="0.1524" layer="91"/>
+</segment>
+</net>
+<net name="N$7" class="0">
+<segment>
+<pinref part="U1" gate="G$1" pin="PB1"/>
+<pinref part="R9" gate="G$1" pin="1"/>
+<wire x1="22.86" y1="20.32" x2="25.4" y2="20.32" width="0.1524" layer="91"/>
+</segment>
+</net>
+<net name="N$5" class="0">
+<segment>
+<pinref part="U1" gate="G$1" pin="PB2"/>
+<pinref part="R8" gate="G$1" pin="1"/>
+<wire x1="22.86" y1="17.78" x2="25.4" y2="17.78" width="0.1524" layer="91"/>
+</segment>
+</net>
+<net name="N$6" class="0">
+<segment>
+<pinref part="U1" gate="G$1" pin="PA7"/>
+<pinref part="R7" gate="G$1" pin="1"/>
+<wire x1="22.86" y1="25.4" x2="25.4" y2="25.4" width="0.1524" layer="91"/>
+</segment>
+</net>
 </nets>
 </sheet>
@@
 </schematic>
 </drawing>
+<compatibility>
+<note version="6.3" minversion="6.2.2" severity="warning">
+Since Version 6.2.2 text objects can contain more than one line,
+which will not be processed correctly with this version.
+</note>
+</compatibility>
 </eagle>

Commit message: redo
Parts:
- J5: value AVRISPWR -> AVRISP0.1"; device dubec:AVRISPWR -> dubec:AVRISP0.1"
Changed lines of the file:
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@@
 <part name="R14" library="dubec" deviceset="RES" device="330_16" value="RES330_16"/>
 <part name="C3" library="dubec" deviceset="CAP" device="47N_50V" value="CAP47N_50V"/>
-<part name="J5" library="dubec" deviceset="AVRISP" device="WR"/>
+<part name="J5" library="dubec" deviceset="AVRISP" device="0.1&quot;" value="AVRISP0.1&quot;"/>
 <part name="R15" library="dubec" deviceset="RES" device="10K_16"/>
 </parts>

Commit message: jack mirror
Connections:
- net !OE: now also J3.3; no longer J3.2
- net +5V: now also J4.2; no longer J4.3
- net +8V: now also J4.1; no longer J4.4
- net BATT-: now also J1.3; no longer J1.2
- net CP: now also J3.2; no longer J3.3
- net DS: now also J3.1; no longer J3.4
- net FB: now also J2.1; no longer J2.4
- net OPTO_A: now also J2.3; no longer J2.2
- net OPTO_C: now also J2.2; no longer J2.3
- net Q7S: now also J1.1; no longer J1.4
- net S+: now also J4.3; no longer J4.2
- net S-: now also J1.4, J2.4, J3.4, J4.4; no longer J1.1, J2.1, J3.1, J4.1
Changed lines of the file:
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@@
 <part name="R3" library="dubec" deviceset="RES" device="330_16" value="RES330_16"/>
 <part name="U1" library="dubec" deviceset="ATTINYX4A" device="8MU"/>
-<part name="J1" library="dubec" deviceset="M04" device="-929P"/>
-<part name="J2" library="dubec" deviceset="M04" device="-929P"/>
-<part name="J3" library="dubec" deviceset="M04" device="-929P"/>
-<part name="J4" library="dubec" deviceset="M04" device="-929P"/>
+<part name="J1" library="dubec" deviceset="M04" device="-929P" value="M04-929P"/>
+<part name="J2" library="dubec" deviceset="M04" device="-929P" value="M04-929P"/>
+<part name="J3" library="dubec" deviceset="M04" device="-929P" value="M04-929P"/>
+<part name="J4" library="dubec" deviceset="M04" device="-929P" value="M04-929P"/>
 <part name="D101" library="dubec" deviceset="LED_DUAL" device="RG-2" value="LED_DUALRG-2"/>
 <part name="D102" library="dubec" deviceset="LED_DUAL" device="RG-2" value="LED_DUALRG-2"/>
@@
 </segment>
 <segment>
-<pinref part="J2" gate="G$1" pin="4"/>
-<wire x1="83.82" y1="15.24" x2="83.82" y2="12.7" width="0.1524" layer="91"/>
-<label x="83.82" y="12.7" size="1.27" layer="95" rot="R270" xref="yes"/>
+<label x="76.2" y="12.7" size="1.27" layer="95" rot="R270" xref="yes"/>
+<wire x1="76.2" y1="15.24" x2="76.2" y2="12.7" width="0.1524" layer="91"/>
+<pinref part="J2" gate="G$1" pin="1"/>
 </segment>
 </net>
@@
 </segment>
 <segment>
-<pinref part="J1" gate="G$1" pin="1"/>
-<wire x1="55.88" y1="15.24" x2="55.88" y2="12.7" width="0.1524" layer="91"/>
-<label x="55.88" y="12.7" size="1.27" layer="95" rot="R270" xref="yes"/>
-</segment>
-<segment>
-<pinref part="J2" gate="G$1" pin="1"/>
-<wire x1="76.2" y1="15.24" x2="76.2" y2="12.7" width="0.1524" layer="91"/>
-<label x="76.2" y="12.7" size="1.27" layer="95" rot="R270" xref="yes"/>
-</segment>
-<segment>
-<pinref part="J3" gate="G$1" pin="1"/>
-<wire x1="83.82" y1="33.02" x2="83.82" y2="35.56" width="0.1524" layer="91"/>
-<label x="83.82" y="35.56" size="1.27" layer="95" rot="R90" xref="yes"/>
-</segment>
-<segment>
-<pinref part="J4" gate="G$1" pin="1"/>
-<wire x1="63.5" y1="33.02" x2="63.5" y2="35.56" width="0.1524" layer="91"/>
-<label x="63.5" y="35.56" size="1.27" layer="95" rot="R90" xref="yes"/>
+<label x="63.5" y="12.7" size="1.27" layer="95" rot="R270" xref="yes"/>
+<wire x1="63.5" y1="15.24" x2="63.5" y2="12.7" width="0.1524" layer="91"/>
+<pinref part="J1" gate="G$1" pin="4"/>
+</segment>
+<segment>
+<label x="83.82" y="12.7" size="1.27" layer="95" rot="R270" xref="yes"/>
+<wire x1="83.82" y1="15.24" x2="83.82" y2="12.7" width="0.1524" layer="91"/>
+<pinref part="J2" gate="G$1" pin="4"/>
+</segment>
+<segment>
+<label x="76.2" y="35.56" size="1.27" layer="95" rot="R90" xref="yes"/>
+<wire x1="76.2" y1="33.02" x2="76.2" y2="35.56" width="0.1524" layer="91"/>
+<pinref part="J3" gate="G$1" pin="4"/>
+</segment>
+<segment>
+<label x="55.88" y="35.56" size="1.27" layer="95" rot="R90" xref="yes"/>
+<wire x1="55.88" y1="33.02" x2="55.88" y2="35.56" width="0.1524" layer="91"/>
+<pinref part="J4" gate="G$1" pin="4"/>
 </segment>
 <segment>
@@
 </segment>
 <segment>
-<pinref part="J2" gate="G$1" pin="2"/>
-<wire x1="78.74" y1="15.24" x2="78.74" y2="12.7" width="0.1524" layer="91"/>
-<label x="78.74" y="12.7" size="1.27" layer="95" rot="R270" xref="yes"/>
+<label x="81.28" y="12.7" size="1.27" layer="95" rot="R270" xref="yes"/>
+<wire x1="81.28" y1="15.24" x2="81.28" y2="12.7" width="0.1524" layer="91"/>
+<pinref part="J2" gate="G$1" pin="3"/>
 </segment>
 </net>
@@
 </segment>
 <segment>
-<pinref part="J2" gate="G$1" pin="3"/>
-<wire x1="81.28" y1="15.24" x2="81.28" y2="12.7" width="0.1524" layer="91"/>
-<label x="81.28" y="12.7" size="1.27" layer="95" rot="R270" xref="yes"/>
+<label x="78.74" y="12.7" size="1.27" layer="95" rot="R270" xref="yes"/>
+<wire x1="78.74" y1="15.24" x2="78.74" y2="12.7" width="0.1524" layer="91"/>
+<pinref part="J2" gate="G$1" pin="2"/>
 </segment>
 </net>
@@
 </segment>
 <segment>
-<pinref part="J4" gate="G$1" pin="3"/>
-<wire x1="58.42" y1="33.02" x2="58.42" y2="35.56" width="0.1524" layer="91"/>
-<label x="58.42" y="35.56" size="1.27" layer="95" rot="R90" xref="yes"/>
+<label x="60.96" y="35.56" size="1.27" layer="95" rot="R90" xref="yes"/>
+<pinref part="J4" gate="G$1" pin="2"/>
+<wire x1="60.96" y1="35.56" x2="60.96" y2="33.02" width="0.1524" layer="91"/>
 </segment>
 <segment>
@@
 <net name="BATT-" class="0">
 <segment>
-<pinref part="J1" gate="G$1" pin="2"/>
-<wire x1="58.42" y1="15.24" x2="58.42" y2="12.7" width="0.1524" layer="91"/>
-<label x="58.42" y="12.7" size="1.27" layer="95" rot="R270" xref="yes"/>
+<label x="60.96" y="12.7" size="1.27" layer="95" rot="R270" xref="yes"/>
+<wire x1="60.96" y1="15.24" x2="60.96" y2="12.7" width="0.1524" layer="91"/>
+<pinref part="J1" gate="G$1" pin="3"/>
 </segment>
 </net>
 <net name="Q7S" class="0">
 <segment>
-<pinref part="J1" gate="G$1" pin="4"/>
-<wire x1="63.5" y1="15.24" x2="63.5" y2="12.7" width="0.1524" layer="91"/>
-<label x="63.5" y="12.7" size="1.27" layer="95" rot="R270" xref="yes"/>
+<label x="55.88" y="12.7" size="1.27" layer="95" rot="R270" xref="yes"/>
+<wire x1="55.88" y1="15.24" x2="55.88" y2="12.7" width="0.1524" layer="91"/>
+<pinref part="J1" gate="G$1" pin="1"/>
 </segment>
 </net>
 <net name="!OE" class="0">
 <segment>
-<pinref part="J3" gate="G$1" pin="2"/>
-<wire x1="81.28" y1="33.02" x2="81.28" y2="35.56" width="0.1524" layer="91"/>
-<label x="81.28" y="35.56" size="1.27" layer="95" rot="R90" xref="yes"/>
+<label x="78.74" y="35.56" size="1.27" layer="95" rot="R90" xref="yes"/>
+<wire x1="78.74" y1="33.02" x2="78.74" y2="35.56" width="0.1524" layer="91"/>
+<pinref part="J3" gate="G$1" pin="3"/>
 </segment>
 <segment>
@@
 <net name="CP" class="0">
 <segment>
-<pinref part="J3" gate="G$1" pin="3"/>
-<wire x1="78.74" y1="33.02" x2="78.74" y2="35.56" width="0.1524" layer="91"/>
-<label x="78.74" y="35.56" size="1.27" layer="95" rot="R90" xref="yes"/>
+<label x="81.28" y="35.56" size="1.27" layer="95" rot="R90" xref="yes"/>
+<wire x1="81.28" y1="33.02" x2="81.28" y2="35.56" width="0.1524" layer="91"/>
+<pinref part="J3" gate="G$1" pin="2"/>
 </segment>
 <segment>
@@
 <net name="DS" class="0">
 <segment>
-<pinref part="J3" gate="G$1" pin="4"/>
-<wire x1="76.2" y1="33.02" x2="76.2" y2="35.56" width="0.1524" layer="91"/>
-<label x="76.2" y="35.56" size="1.27" layer="95" rot="R90" xref="yes"/>
+<label x="83.82" y="35.56" size="1.27" layer="95" rot="R90" xref="yes"/>
+<wire x1="83.82" y1="33.02" x2="83.82" y2="35.56" width="0.1524" layer="91"/>
+<pinref part="J3" gate="G$1" pin="1"/>
 </segment>
 <segment>
@@
 <net name="S+" class="0">
 <segment>
-<pinref part="J4" gate="G$1" pin="2"/>
-<wire x1="60.96" y1="33.02" x2="60.96" y2="35.56" width="0.1524" layer="91"/>
-<label x="60.96" y="35.56" size="1.27" layer="95" rot="R90" xref="yes"/>
+<label x="58.42" y="35.56" size="1.27" layer="95" rot="R90" xref="yes"/>
+<pinref part="J4" gate="G$1" pin="3"/>
+<wire x1="58.42" y1="35.56" x2="58.42" y2="33.02" width="0.1524" layer="91"/>
 </segment>
 <segment>
@@
 <net name="+8V" class="0">
 <segment>
-<pinref part="J4" gate="G$1" pin="4"/>
-<wire x1="55.88" y1="33.02" x2="55.88" y2="35.56" width="0.1524" layer="91"/>
-<label x="55.88" y="35.56" size="1.27" layer="95" rot="R90" xref="yes"/>
-</segment>
-<segment>
+<label x="63.5" y="35.56" size="1.27" layer="95" rot="R90" xref="yes"/>
+<wire x1="63.5" y1="33.02" x2="63.5" y2="35.56" width="0.1524" layer="91"/>
+<pinref part="J4" gate="G$1" pin="1"/>
+</segment>
+<segment>
