File: lipovsky-control.brd (EAGLE design)
At the start: 59 x 32 mm, 44 parts, among them J5 AVRISP0.1", P1 M04-929P, P2 M04-929P, P3 M04-929P, P4 M04-929P, U1 ATTINYX4A8MU, U2 MIC2288YD5, U3 MIC2288YD5, U7 LTV-816S

Commit message: .
Parts:
- renumbered U7 to U4
Changed lines of the file:
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@@
 <attribute name="FLASH" value="8KB (4K x 16)" x="20" y="23" size="1.778" layer="27" rot="R180" display="off"/>
 </element>
-<element name="U7" library="dubec" package="4-OPTO-1" value="LTV-816S" x="32" y="17" rot="R90">
+<element name="U4" library="dubec" package="4-OPTO-1" value="LTV-816S" x="32" y="17" rot="R90">
 <attribute name="DIGIKEY_PART_#" value="160-1361-5-ND" x="32" y="17" size="1.778" layer="27" rot="R90" display="off"/>
 <attribute name="TEMP" value="-50°C ~ 110°C" x="32" y="17" size="1.778" layer="27" rot="R90" display="off"/>
@@
 <signals>
 <signal name="FB">
-<contactref element="U7" pad="3"/>
+<contactref element="U4" pad="3"/>
 <contactref element="R3" pad="2"/>
 <contactref element="R14" pad="2"/>
@@
 </signal>
 <signal name="OPTO_A">
-<contactref element="U7" pad="1"/>
+<contactref element="U4" pad="1"/>
 <wire x1="45.43" y1="3.3" x2="36.8" y2="3.3" width="0.3" layer="1"/>
 <wire x1="36.8" y1="3.3" x2="36" y2="4.1" width="0.3" layer="1"/>
@@
 </signal>
 <signal name="OPTO_C">
-<contactref element="U7" pad="2"/>
+<contactref element="U4" pad="2"/>
 <via x="36.5" y="17.1" extent="1-16" drill="0.35"/>
 <wire x1="36.5" y1="18.27" x2="36.5" y2="17.1" width="0.6" layer="1"/>
@@
 <wire x1="27.95" y1="26.1" x2="27.95" y2="24.95" width="0.6" layer="1"/>
 <contactref element="R12" pad="1"/>
-<contactref element="U7" pad="4"/>
+<contactref element="U4" pad="4"/>
 <contactref element="C1" pad="2"/>
 <contactref element="R15" pad="1"/>

Commit message: tweaks
Changed lines of the file:
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@@
 <attribute name="EBAY_PART_#" value="3296W-502" x="32" y="13" size="1.778" layer="27" display="off"/>
 <attribute name="DIGIKEY_PART_#" value="3296W-502-ND" x="32" y="13" size="1.778" layer="27" display="off"/>
+<attribute name="EPK" value="78.80" x="32" y="13" size="1.778" layer="27" display="off"/>
 </element>
 <element name="R3" library="dubec" package="0402" value="RES330_16" x="29.65" y="19.8" rot="R180">
@@
 <attribute name="TEMP" value="-40°C ~ 85°C (TA)" x="20" y="23" size="1.778" layer="27" rot="R180" display="off"/>
 <attribute name="MANUFACTURER" value="Atmel" x="20" y="23" size="1.778" layer="27" rot="R180" display="off"/>
-<attribute name="EURO" value="637.90/1000" x="20" y="23" size="1.778" layer="27" rot="R180" display="off"/>
 <attribute name="MFG_PART_#" value="ATTINY84A-MU" x="20" y="23" size="1.778" layer="27" rot="R180" display="off"/>
 <attribute name="ADC" value="8x10b" x="20" y="23" size="1.778" layer="27" rot="R180" display="off"/>
 <attribute name="FLASH" value="8KB (4K x 16)" x="20" y="23" size="1.778" layer="27" rot="R180" display="off"/>
+<attribute name="EPK" value="636.98" x="20" y="23" size="1.778" layer="27" rot="R180" display="off"/>
 </element>
 <element name="U4" library="dubec" package="4-OPTO-1" value="LTV-816S" x="32" y="17" rot="R90">
@@
 <attribute name="MANUFACTURER" value="Lite-On Inc." x="32" y="17" size="1.778" layer="27" rot="R90" display="off"/>
 <attribute name="I_FWD" value="50mA" x="32" y="17" size="1.778" layer="27" rot="R90" display="off"/>
-<attribute name="EURO" value="5.67/25" x="32" y="17" size="1.778" layer="27" rot="R90" display="off"/>
 <attribute name="MFG_PART_#" value="LTV-816S" x="32" y="17" size="1.778" layer="27" rot="R90" display="off"/>
+<attribute name="EPK" value="101.94" x="32" y="17" size="1.778" layer="27" rot="R90" display="off"/>
 </element>
 <element name="P1" library="dubec" package="1X04_929P" value="M04-929P" x="20" y="2" rot="MR0">
@@
 <attribute name="V_FWD" value="480mV @ 500mA" x="27.95" y="26.8" size="1.778" layer="27" rot="R270" display="off"/>
 <attribute name="MANUFACTURER" value="ON Semiconductor" x="27.95" y="26.8" size="1.778" layer="27" rot="R270" display="off"/>
-<attribute name="EURO" value="3.13/10" x="27.95" y="26.8" size="1.778" layer="27" rot="R270" display="off"/>
+<attribute name="EPK" value="85.82" x="27.95" y="26.8" size="1.778" layer="27" rot="R270" display="off"/>
 </element>
 <element name="D3" library="dubec" package="SOD523+" value="D_SCH20V_0.5A" x="33.55" y="26.8" rot="R270">
@@
 <attribute name="V_FWD" value="480mV @ 500mA" x="33.55" y="26.8" size="1.778" layer="27" rot="R270" display="off"/>
 <attribute name="MANUFACTURER" value="ON Semiconductor" x="33.55" y="26.8" size="1.778" layer="27" rot="R270" display="off"/>
-<attribute name="EURO" value="3.13/10" x="33.55" y="26.8" size="1.778" layer="27" rot="R270" display="off"/>
+<attribute name="EPK" value="85.82" x="33.55" y="26.8" size="1.778" layer="27" rot="R270" display="off"/>
 </element>
 <element name="R2" library="dubec" package="0402" value="RES14.3K_16" x="30.5" y="24.7" rot="R270">
@@
 <element name="R15" library="dubec" package="0402" value="RES10K_16" x="14.9" y="26.725" rot="R180">
 <attribute name="MANUFACTURER" value="Vishay Dale" x="14.9" y="26.725" size="1.778" layer="27" rot="R180" display="off"/>
-<attribute name="EURO" value="2.10/50" x="14.9" y="26.725" size="1.778" layer="27" rot="R180" display="off"/>
 <attribute name="MFG_PART_#" value="CRCW040210K0FKED" x="14.9" y="26.725" size="1.778" layer="27" rot="R180" display="off"/>
 <attribute name="DIGIKEY_PART_#" value="541-10.0KLCT-ND" x="14.9" y="26.725" size="1.778" layer="27" rot="R180" display="off"/>
 <attribute name="TEMP" value="±100ppm/°C" x="14.9" y="26.725" size="1.778" layer="27" rot="R180" display="off"/>
 <attribute name="TOLERANCE" value="±1%" x="14.9" y="26.725" size="1.778" layer="27" rot="R180" display="off"/>
+<attribute name="EPK" value="5.24" x="14.9" y="26.725" size="1.778" layer="27" rot="R180" display="off"/>
 </element>
 <element name="U$1" library="dubec" package="TF-EMBLEM" value="" x="15" y="16" rot="R90"/>
@@
 <wire x1="29.15" y1="19.8" x2="29.15" y2="18.875" width="0.4" layer="1"/>
 <wire x1="26.3" y1="20.5" x2="26.45" y2="20.35" width="0.3" layer="1"/>
-<wire x1="26.45" y1="20.35" x2="26.45" y2="19.125" width="0.3" layer="1"/>
-<wire x1="26.45" y1="19.125" x2="26.7" y2="18.875" width="0.3" layer="1"/>
-<wire x1="26.7" y1="18.875" x2="26.895" y2="18.875" width="0.3" layer="1"/>
-<wire x1="26.895" y1="18.875" x2="27.5" y2="18.27" width="0.3" layer="1"/>
+<wire x1="26.45" y1="20.35" x2="26.45" y2="19.32" width="0.3" layer="1"/>
 <wire x1="29.15" y1="16.25" x2="30.7" y2="14.7" width="0.3" layer="16"/>
 <wire x1="30.7" y1="14.7" x2="30.7" y2="12.4" width="0.3" layer="16"/>
 <wire x1="29.15" y1="16.25" x2="29.15" y2="18.875" width="0.3" layer="16"/>
+<wire x1="27.5" y1="18.27" x2="26.45" y2="19.32" width="0.3" layer="1"/>
 </signal>
 <signal name="S-">
@@
 <wire x1="27.1" y1="14.4" x2="27.2" y2="14.5" width="0.3" layer="16"/>
 <via x="17.6" y="21.1" extent="1-16" drill="0.35"/>
-<wire x1="19.46" y1="18.27" x2="19.46" y2="19.24" width="0.3" layer="1"/>
-<wire x1="19.46" y1="19.24" x2="17.6" y2="21.1" width="0.3" layer="1"/>
 <wire x1="17.6" y1="21.1" x2="17.6" y2="28.87" width="0.3" layer="16"/>
 <wire x1="15.4" y1="26.725" x2="15.65" y2="26.975" width="0.3" layer="1"/>
@@
 <wire x1="18.73" y1="27.97" x2="18.73" y2="30" width="0.7" layer="1"/>
 <wire x1="17.6" y1="28.87" x2="18.73" y2="30" width="0.3" layer="16"/>
+<wire x1="19.46" y1="18.27" x2="18.7" y2="19.03" width="0.3" layer="1"/>
+<wire x1="18.7" y1="19.03" x2="18.7" y2="20" width="0.3" layer="1"/>
+<wire x1="18.7" y1="20" x2="17.6" y2="21.1" width="0.3" layer="1"/>
 </signal>
 <signal name="BATT-">
@@
 <contactref element="J5" pad="1"/>
 <contactref element="P3" pad="2"/>
-<wire x1="21" y1="21.1" x2="21" y2="19.1" width="0.25" layer="1"/>
-<wire x1="21" y1="19.1" x2="20.725" y2="18.825" width="0.25" layer="1"/>
-<wire x1="20.725" y1="18.825" x2="20.725" y2="16.995" width="0.25" layer="1"/>
+<wire x1="21" y1="21.1" x2="21" y2="19.2" width="0.25" layer="1"/>
+<wire x1="21" y1="19.2" x2="20.725" y2="18.925" width="0.25" layer="1"/>
+<wire x1="20.725" y1="18.925" x2="20.725" y2="16.995" width="0.25" layer="1"/>
 <wire x1="20.725" y1="16.995" x2="19.46" y2="15.73" width="0.25" layer="1"/>
 <wire x1="45.43" y1="28.7" x2="42.4" y2="28.7" width="0.3" layer="16"/>

Commit message: tidy
Parts:
- moved R3 0.40 mm to (29.6, 20.2)
Changed lines of the file:
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@@
 <attribute name="EPK" value="78.80" x="32" y="13" size="1.778" layer="27" display="off"/>
 </element>
-<element name="R3" library="dubec" package="0402" value="RES330_16" x="29.65" y="19.8" rot="R180">
-<attribute name="DIGIKEY_PART_#" value="541-330LCT-ND" x="29.65" y="19.8" size="1.778" layer="27" rot="R180" display="off"/>
-<attribute name="TEMP" value="±100ppm/°C" x="29.65" y="19.8" size="1.778" layer="27" rot="R180" display="off"/>
-<attribute name="MANUFACTURER" value="Vishay Dale" x="29.65" y="19.8" size="1.778" layer="27" rot="R180" display="off"/>
-<attribute name="MFG_PART_#" value="CRCW0402330RFKED" x="29.65" y="19.8" size="1.778" layer="27" rot="R180" display="off"/>
-<attribute name="TOLERANCE" value="±1%" x="29.65" y="19.8" size="1.778" layer="27" rot="R180" display="off"/>
-<attribute name="EPK" value="5.24" x="29.65" y="19.8" size="1.778" layer="27" rot="R180" display="off"/>
+<element name="R3" library="dubec" package="0402" value="RES330_16" x="29.65" y="20.2" rot="R180">
+<attribute name="DIGIKEY_PART_#" value="541-330LCT-ND" x="29.65" y="20.2" size="1.778" layer="27" rot="R180" display="off"/>
+<attribute name="TEMP" value="±100ppm/°C" x="29.65" y="20.2" size="1.778" layer="27" rot="R180" display="off"/>
+<attribute name="MANUFACTURER" value="Vishay Dale" x="29.65" y="20.2" size="1.778" layer="27" rot="R180" display="off"/>
+<attribute name="MFG_PART_#" value="CRCW0402330RFKED" x="29.65" y="20.2" size="1.778" layer="27" rot="R180" display="off"/>
+<attribute name="TOLERANCE" value="±1%" x="29.65" y="20.2" size="1.778" layer="27" rot="R180" display="off"/>
+<attribute name="EPK" value="5.24" x="29.65" y="20.2" size="1.778" layer="27" rot="R180" display="off"/>
 </element>
 <element name="U1" library="dubec" package="ATTINYX4A" value="ATTINYX4A8MU" x="20" y="23" rot="R180">
@@
 <wire x1="27.5" y1="18.27" x2="28.105" y2="18.875" width="0.3" layer="1"/>
 <wire x1="28.105" y1="18.875" x2="29.15" y2="18.875" width="0.3" layer="1"/>
-<wire x1="29.15" y1="19.8" x2="29.15" y2="18.875" width="0.4" layer="1"/>
+<wire x1="29.15" y1="20.2" x2="29.15" y2="18.875" width="0.4" layer="1"/>
 <wire x1="26.3" y1="20.5" x2="26.45" y2="20.35" width="0.3" layer="1"/>
 <wire x1="26.45" y1="20.35" x2="26.45" y2="19.32" width="0.3" layer="1"/>
@@
 <wire x1="17.99" y1="3.8" x2="35.4" y2="3.8" width="0.3" layer="1"/>
 <wire x1="35.4" y1="10.84" x2="35.4" y2="3.8" width="0.3" layer="1"/>
-<via x="19.2" y="23.7" extent="1-16" drill="0.4"/>
+<via x="19.2" y="23.7" extent="1-16" drill="0.35"/>
 <polygon width="0.2" layer="16" isolate="0.25" thermals="no">
 <vertex x="18" y="21.7"/>
@@
 </polygon>
 <wire x1="43.49" y1="2.7" x2="44.19" y2="2" width="0.3" layer="1"/>
-<via x="20.8" y="23.7" extent="1-16" drill="0.4"/>
+<via x="20.8" y="23.7" extent="1-16" drill="0.35"/>
 <wire x1="20" y1="24.9" x2="20" y2="23" width="0.25" layer="1"/>
 <wire x1="24.6" y1="22.7" x2="25.3" y2="22.7" width="0.4" layer="1"/>
@@
 <wire x1="24.54" y1="20.5" x2="24.8" y2="20.5" width="0.3" layer="1"/>
 <wire x1="27.7" y1="30" x2="30" y2="27.7" width="0.8" layer="16"/>
-<via x="23.1" y="26.6" extent="1-16" drill="0.4"/>
+<via x="23.1" y="26.6" extent="1-16" drill="0.35"/>
 <wire x1="23.1" y1="26.6" x2="24" y2="26.6" width="0.7" layer="1"/>
 <wire x1="20.5" y1="26.5" x2="20.6" y2="26.6" width="0.7" layer="1"/>
@@
 <wire x1="25.2" y1="27.175" x2="24.675" y2="27.7" width="0.7" layer="1"/>
 <wire x1="24.675" y1="27.7" x2="19" y2="27.7" width="0.7" layer="1"/>
-<wire x1="27.95" y1="26.1" x2="26.9" y2="26.1" width="0.6" layer="1"/>
-<wire x1="26.9" y1="26.1" x2="26.45" y2="26.55" width="0.6" layer="1"/>
-<wire x1="26.45" y1="26.55" x2="25.35" y2="26.55" width="0.6" layer="1"/>
+<wire x1="27.95" y1="26.1" x2="27.4" y2="26.1" width="0.6" layer="1"/>
+<wire x1="27.4" y1="26.1" x2="26.95" y2="26.55" width="0.6" layer="1"/>
+<wire x1="26.95" y1="26.55" x2="25.35" y2="26.55" width="0.6" layer="1"/>
 <wire x1="25.35" y1="26.55" x2="25.3" y2="26.6" width="0.6" layer="1"/>
 <wire x1="19" y1="27.7" x2="18.73" y2="27.97" width="0.7" layer="1"/>
@@
 <via x="20.2" y="19.6" extent="1-16" drill="0.35"/>
 <wire x1="19" y1="21.1" x2="19" y2="20.6" width="0.25" layer="1"/>
-<wire x1="19" y1="20.6" x2="20" y2="19.6" width="0.25" layer="1"/>
-<wire x1="20" y1="19.6" x2="20.2" y2="19.6" width="0.25" layer="1"/>
+<wire x1="19" y1="20.6" x2="19.2" y2="20.4" width="0.25" layer="1"/>
+<wire x1="19.2" y1="20.4" x2="19.9" y2="20.4" width="0.25" layer="1"/>
+<wire x1="19.9" y1="20.4" x2="20.2" y2="20.1" width="0.25" layer="1"/>
+<wire x1="20.2" y1="20.1" x2="20.2" y2="19.6" width="0.25" layer="1"/>
 <wire x1="20.67" y1="19.6" x2="22" y2="18.27" width="0.3" layer="16"/>
 <wire x1="26.7" y1="20.2" x2="30" y2="23.5" width="0.3" layer="16"/>
@@
 <contactref element="D5" pad="C1"/>
 <contactref element="D5" pad="A2"/>
-<via x="23.175" y="25.1" extent="1-16" drill="0.35"/>
-<wire x1="23.175" y1="25.1" x2="23.175" y2="24.375" width="0.3" layer="16"/>
-<wire x1="23.175" y1="24.375" x2="20.4" y2="21.6" width="0.3" layer="16"/>
+<via x="23.1" y="25.1" extent="1-16" drill="0.35"/>
+<wire x1="23.1" y1="25.1" x2="23.1" y2="24.3" width="0.3" layer="16"/>
+<wire x1="23.1" y1="24.3" x2="20.4" y2="21.6" width="0.3" layer="16"/>
 <wire x1="20.4" y1="21.6" x2="19.2" y2="21.6" width="0.3" layer="16"/>
 <wire x1="19.2" y1="21.6" x2="16.3" y2="18.7" width="0.3" layer="16"/>
@@
 <wire x1="19.15" y1="6.95" x2="19.15" y2="7.65" width="0.3" layer="1"/>
 <wire x1="19.15" y1="7.65" x2="19" y2="7.8" width="0.3" layer="1"/>
-<wire x1="23.175" y1="25.1" x2="24" y2="25.1" width="0.7" layer="1"/>
+<wire x1="23.1" y1="25.1" x2="24" y2="25.1" width="0.7" layer="1"/>
 <wire x1="24" y1="25.1" x2="25.3" y2="25.1" width="0.7" layer="1"/>
 </signal>
@@
 <contactref element="R3" pad="1"/>
 <contactref element="R1" pad="WIPER"/>
-<wire x1="30.2" y1="16.1" x2="30.2" y2="19.75" width="0.3" layer="1"/>
-<wire x1="30.2" y1="19.75" x2="30.15" y2="19.8" width="0.3" layer="1"/>
+<wire x1="30.2" y1="16.1" x2="30.2" y2="20.15" width="0.3" layer="1"/>
+<wire x1="30.2" y1="20.15" x2="30.15" y2="20.2" width="0.3" layer="1"/>
 <wire x1="30.2" y1="16.1" x2="32" y2="14.3" width="0.3" layer="1"/>
 <wire x1="32" y1="14.3" x2="32" y2="13" width="0.3" layer="1"/>

Commit message: power mcu
Parts:
- U1: device dubec:ATTINYX4A -> dubec:20M1
Changed lines of the file:
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@@
 <attribute name="EPK" value="5.24" x="29.65" y="20.2" size="1.778" layer="27" rot="R180" display="off"/>
 </element>
-<element name="U1" library="dubec" package="ATTINYX4A" value="ATTINYX4A8MU" x="20" y="23" rot="R180">
+<element name="U1" library="dubec" package="20M1" value="ATTINYX4A8MU" x="20" y="23" rot="R180">
 <attribute name="FREQ" value="20MHz" x="20" y="23" size="1.778" layer="27" rot="R180" display="off"/>
 <attribute name="RAM" value="512 x 8" x="20" y="23" size="1.778" layer="27" rot="R180" display="off"/>
@@
 <attribute name="MFG_PART_#" value="ATTINY84A-MU" x="20" y="23" size="1.778" layer="27" rot="R180" display="off"/>
 <attribute name="ADC" value="8x10b" x="20" y="23" size="1.778" layer="27" rot="R180" display="off"/>
-<attribute name="FLASH" value="8KB (4K x 16)" x="20" y="23" size="1.778" layer="27" rot="R180" display="off"/>
+<attribute name="FLASH" value="4K x 16" x="20" y="23" size="1.778" layer="27" rot="R180" display="off"/>
 <attribute name="EPK" value="636.98" x="20" y="23" size="1.778" layer="27" rot="R180" display="off"/>
 </element>
